Commit message: thumb fix

File: ros2_ws/src/prosthesis_description/model/parameters.xacro (robot description, xacro)
@@ -31,5 +31,5 @@
     <xacro:property name="little_middle_width" value="0.015" />
     <xacro:property name="little_middle_depth" value="0.012" />
-    <xacro:property name="thumb_metacarpal_length" value="0.028" />
+    <xacro:property name="thumb_metacarpal_length" value="0.01" />
     <xacro:property name="thumb_metacarpal_width" value="0.015" />
     <xacro:property name="thumb_metacarpal_depth" value="0.012" />

File: ros2_ws/src/prosthesis_description/model/prosthesis.urdf.xacro (robot description, xacro)
@@ -164,4 +164,8 @@
         <geometry><box size="${thumb_metacarpal_length} ${thumb_metacarpal_width} ${thumb_metacarpal_depth}"/></geometry>
     </visual>
+    <collision>
+        <origin xyz="${thumb_metacarpal_length/2} 0 0" rpy="0 0 0"/>
+        <geometry><box size="${thumb_metacarpal_length} ${thumb_metacarpal_width} ${thumb_metacarpal_depth}"/></geometry>
+    </collision>
     <xacro:inertial_box mass="0.01" x="${thumb_metacarpal_length}" y="${thumb_metacarpal_width}" z="${thumb_metacarpal_depth}">
         <origin xyz="${thumb_metacarpal_length/2} 0 0" rpy="0 0 0"/>
@@ -173,4 +177,8 @@
         <geometry><box size="${thumb_proximal_length} ${thumb_proximal_width} ${thumb_proximal_depth}"/></geometry>
     </visual>
+    <collision>
+        <origin xyz="${thumb_proximal_length/2} 0 0" rpy="0 0 0"/>
+        <geometry><box size="${thumb_proximal_length} ${thumb_proximal_width} ${thumb_proximal_depth}"/></geometry>
+    </collision>
     <xacro:inertial_box mass="0.01" x="${thumb_proximal_length}" y="${thumb_proximal_width}" z="${thumb_proximal_depth}">
         <origin xyz="${thumb_proximal_length/2} 0 0" rpy="0 0 0"/>
@@ -258,5 +266,5 @@
   <joint name="joint_thumb_cmc" type="revolute">
     <parent link="palm_link"/><child link="thumb_metacarpal_link"/>
-    <origin xyz="${thumb_metacarpal_width/2} ${-(palm_width/2.5)} 0.00" rpy="0 0 -0.70"/><axis xyz="0 1 0"/>
+    <origin xyz="${thumb_metacarpal_width/2 + 0.02} ${-(palm_width/2) - 0.0068} 0.00" rpy="0 0 -0.80"/><axis xyz="0 1 0"/>
     <limit lower="-0.40" upper="1.20" effort="3" velocity="5"/>
   </joint>
