Commit message: Gazebo spawn tentative : creation of prosthesis.gazebo, creation of gazebo.launch.py

File: ros2_ws/src/prosthesis_description/model/prosthesis.urdf.xacro (robot description, xacro)
@@ -2,4 +2,5 @@
 <robot xmlns:xacro="http://www.ros.org/wiki/xacro" name="hand">
 <xacro:include filename="useful_tags.xacro" />
+<xacro:include filename="prosthesis.gazebo" />
   <!-- ===== LINKS (base & palm unchanged) ===== -->
   <link name="world" />
@@ -194,5 +195,5 @@
     <collision>
         <origin xyz="${thumb_metacarpal_length/2} 0 0" rpy="0 0 0"/>
-        <geometry><box size="${thumb_metacarpal_length} ${thumb_metacarpal_width} ${thumb_metacarpal_depth}"/></geometry>
+        <geometry><box size="0 0 0"/></geometry>
     </collision>
     <xacro:inertial_box mass="0.01" x="${thumb_metacarpal_length}" y="${thumb_metacarpal_width}" z="${thumb_metacarpal_depth}">

Commit message: First changes for ros2_control integration (#4)

File: ros2_ws/src/prosthesis_description/model/prosthesis.urdf.xacro (robot description, xacro)
@@ -1,10 +1,8 @@
 <?xml version="1.0"?>
 <robot xmlns:xacro="http://www.ros.org/wiki/xacro" name="hand">
-<xacro:include filename="useful_tags.xacro" />
+<xacro:include filename="parameters.xacro" />
+<xacro:include filename="gazebo.xacro" />
   <!-- ===== LINKS (base & palm unchanged) ===== -->
   <link name="world" />
-  <xacro:property name="base_length" value="0.174" />
-  <xacro:property name="base_width" value="0.065" />
-  <xacro:property name="base_depth" value="0.101" />
   <link name="base_link">
     <visual>
@@ -34,7 +32,4 @@
     </xacro:inertial_sphere>
   </link>
-  <xacro:property name="palm_length" value="0.068" />
-  <xacro:property name="palm_width" value="0.098" />
-  <xacro:property name="palm_depth" value="0.019" />
   <link name="palm_link">
     <visual>
@@ -52,7 +47,4 @@
   <!-- ===== FINGER & THUMB LINKS (all boxes 0.02 x 0.05 x 0.02) ===== -->
   <!-- Index -->
-  <xacro:property name="index_proximal_length" value="0.025" />
-  <xacro:property name="index_proximal_width" value="0.015" />
-  <xacro:property name="index_proximal_depth" value="0.012" />
   <link name="index_proximal_link">
     <visual>
@@ -68,7 +60,4 @@
     </xacro:inertial_box>
   </link>
-  <xacro:property name="index_middle_length" value="0.05" />
-  <xacro:property name="index_middle_width" value="0.015" />
-  <xacro:property name="index_middle_depth" value="0.012" />
   <link name="index_middle_link">
     <visual>
@@ -85,7 +74,4 @@
   </link>
   <!-- Middle -->
-  <xacro:property name="middle_proximal_length" value="0.025" />
-  <xacro:property name="middle_proximal_width" value="0.015" />
-  <xacro:property name="middle_proximal_depth" value="0.012" />
   <link name="middle_proximal_link">
     <visual>
@@ -118,7 +104,4 @@
   </link>
   <!-- Ring -->
-  <xacro:property name="ring_proximal_length" value="0.025" />
-  <xacro:property name="ring_proximal_width" value="0.015" />
-  <xacro:property name="ring_proximal_depth" value="0.012" />
   <link name="ring_proximal_link">
     <visual>
@@ -134,7 +117,4 @@
     </xacro:inertial_box>
   </link>
-  <xacro:property name="ring_middle_length" value="0.05" />
-  <xacro:property name="ring_middle_width" value="0.015" />
-  <xacro:property name="ring_middle_depth" value="0.012" />
   <link name="ring_middle_link">
     <visual>
@@ -151,7 +131,4 @@
   </link>
   <!-- Little -->
-  <xacro:property name="little_proximal_length" value="0.025" />
-  <xacro:property name="little_proximal_width" value="0.015" />
-  <xacro:property name="little_proximal_depth" value="0.012" />
   <link name="little_proximal_link">
     <visual>
@@ -167,7 +144,4 @@
     </xacro:inertial_box>
   </link>
-  <xacro:property name="little_middle_length" value="0.05" />
-  <xacro:property name="little_middle_width" value="0.015" />
-  <xacro:property name="little_middle_depth" value="0.012" />
   <link name="little_middle_link">
     <visual>
@@ -184,7 +158,4 @@
   </link>
   <!-- Thumb -->
-  <xacro:property name="thumb_metacarpal_length" value="0.028" />
-  <xacro:property name="thumb_metacarpal_width" value="0.015" />
-  <xacro:property name="thumb_metacarpal_depth" value="0.012" />
   <link name="thumb_metacarpal_link">
     <visual>
@@ -194,5 +165,5 @@
     <collision>
         <origin xyz="${thumb_metacarpal_length/2} 0 0" rpy="0 0 0"/>
-        <geometry><box size="${thumb_metacarpal_length} ${thumb_metacarpal_width} ${thumb_metacarpal_depth}"/></geometry>
+        <geometry><box size="0 0 0"/></geometry>
     </collision>
     <xacro:inertial_box mass="0.01" x="${thumb_metacarpal_length}" y="${thumb_metacarpal_width}" z="${thumb_metacarpal_depth}">
@@ -200,7 +171,4 @@
     </xacro:inertial_box>
   </link>
-  <xacro:property name="thumb_proximal_length" value="0.025" />
-  <xacro:property name="thumb_proximal_width" value="0.015" />
-  <xacro:property name="thumb_proximal_depth" value="0.012" />
   <link name="thumb_proximal_link">
     <visual>
@@ -216,7 +184,4 @@
     </xacro:inertial_box>
   </link>
-  <xacro:property name="thumb_distal_length" value="0.020" />
-  <xacro:property name="thumb_distal_width" value="0.015" />
-  <xacro:property name="thumb_distal_depth" value="0.012" />
   <link name="thumb_distal_link">
     <visual>
@@ -253,13 +218,4 @@
     <limit lower="-1.57" upper="1.57" effort="5" velocity="5"/>
   </joint>
-  <!-- MCP X and Y positions for each finger relative to palm_link -->
-  <xacro:property name="mcp_x" value="${palm_length}" />
-  <xacro:property name="finger_width" value="${index_proximal_length}" />
-  <xacro:property name="spacing_area" value="${palm_width - finger_width * 4}"/>
-  <xacro:property name="d" value="${spacing_area / 5}"/>
-  <xacro:property name="index_mcp_y" value="${-palm_width / 2 + d + finger_width / 2}" />
-  <xacro:property name="middle_mcp_y" value="${-palm_width / 2 + d*2 + finger_width*1.5}" />
-  <xacro:property name="ring_mcp_y" value="${-palm_width / 2 + d*3 + finger_width*2.5}" />
-  <xacro:property name="little_mcp_y" value="${-palm_width / 2 + d*4 + finger_width*3.5}" />
   <!-- Index -->
   <joint name="joint_index_mcp" type="revolute">

Commit message: - Added scripts : joint_state_printer.py and movement_input.py -  Added joint_trajectory_controller - Added own empty world - Thumb collisions are not correct but they'll change with the meca meshes anyway

File: ros2_ws/src/prosthesis_description/model/prosthesis.urdf.xacro (robot description, xacro)
@@ -164,8 +164,4 @@
         <geometry><box size="${thumb_metacarpal_length} ${thumb_metacarpal_width} ${thumb_metacarpal_depth}"/></geometry>
     </visual>
-    <collision>
-        <origin xyz="${thumb_metacarpal_length/2} 0 0" rpy="0 0 0"/>
-        <geometry><box size="0 0 0"/></geometry>
-    </collision>
     <xacro:inertial_box mass="0.01" x="${thumb_metacarpal_length}" y="${thumb_metacarpal_width}" z="${thumb_metacarpal_depth}">
         <origin xyz="${thumb_metacarpal_length/2} 0 0" rpy="0 0 0"/>
@@ -177,8 +173,4 @@
         <geometry><box size="${thumb_proximal_length} ${thumb_proximal_width} ${thumb_proximal_depth}"/></geometry>
     </visual>
-    <collision>
-        <origin xyz="${thumb_proximal_length/2} 0 0" rpy="0 0 0"/>
-        <geometry><box size="${thumb_proximal_length} ${thumb_proximal_width} ${thumb_proximal_depth}"/></geometry>
-    </collision>
     <xacro:inertial_box mass="0.01" x="${thumb_proximal_length}" y="${thumb_proximal_width}" z="${thumb_proximal_depth}">
         <origin xyz="${thumb_proximal_length/2} 0 0" rpy="0 0 0"/>

Commit message: basic ros2 control (#5)
added Gazebo-ros plugins

added basic controllers : Use of joint_state_broadcaster which can publish the state of the registered hardware interfaces and joint_trajectory_controller which can create an action when receiving a trajectory for the robot to execute.

implemented script movement_input.py which can send a trajectory to the joint_trajectory_controller. When run we see the prosthesis move in gz simulation.

implemented script joint_state_printer.py which subscribes to the topic /joint_states and prints infos for each joint.

File: ros2_ws/src/prosthesis_description/model/prosthesis.urdf.xacro (robot description, xacro)
@@ -1,10 +1,9 @@
 <?xml version="1.0"?>
 <robot xmlns:xacro="http://www.ros.org/wiki/xacro" name="hand">
-<xacro:include filename="useful_tags.xacro" />
+<!--File containing all the fundamental links and joints description-->
+<xacro:include filename="parameters.xacro" />
+<xacro:include filename="gazebo.xacro" />
   <!-- ===== LINKS (base & palm unchanged) ===== -->
   <link name="world" />
-  <xacro:property name="base_length" value="0.174" />
-  <xacro:property name="base_width" value="0.065" />
-  <xacro:property name="base_depth" value="0.101" />
   <link name="base_link">
     <visual>
@@ -34,7 +33,4 @@
     </xacro:inertial_sphere>
   </link>
-  <xacro:property name="palm_length" value="0.068" />
-  <xacro:property name="palm_width" value="0.098" />
-  <xacro:property name="palm_depth" value="0.019" />
   <link name="palm_link">
     <visual>
@@ -52,7 +48,4 @@
   <!-- ===== FINGER & THUMB LINKS (all boxes 0.02 x 0.05 x 0.02) ===== -->
   <!-- Index -->
-  <xacro:property name="index_proximal_length" value="0.025" />
-  <xacro:property name="index_proximal_width" value="0.015" />
-  <xacro:property name="index_proximal_depth" value="0.012" />
   <link name="index_proximal_link">
     <visual>
@@ -68,7 +61,4 @@
     </xacro:inertial_box>
   </link>
-  <xacro:property name="index_middle_length" value="0.05" />
-  <xacro:property name="index_middle_width" value="0.015" />
-  <xacro:property name="index_middle_depth" value="0.012" />
   <link name="index_middle_link">
     <visual>
@@ -85,7 +75,4 @@
   </link>
   <!-- Middle -->
-  <xacro:property name="middle_proximal_length" value="0.025" />
-  <xacro:property name="middle_proximal_width" value="0.015" />
-  <xacro:property name="middle_proximal_depth" value="0.012" />
   <link name="middle_proximal_link">
     <visual>
@@ -118,7 +105,4 @@
   </link>
   <!-- Ring -->
-  <xacro:property name="ring_proximal_length" value="0.025" />
-  <xacro:property name="ring_proximal_width" value="0.015" />
-  <xacro:property name="ring_proximal_depth" value="0.012" />
   <link name="ring_proximal_link">
     <visual>
@@ -134,7 +118,4 @@
     </xacro:inertial_box>
   </link>
-  <xacro:property name="ring_middle_length" value="0.05" />
-  <xacro:property name="ring_middle_width" value="0.015" />
-  <xacro:property name="ring_middle_depth" value="0.012" />
   <link name="ring_middle_link">
     <visual>
@@ -151,7 +132,4 @@
   </link>
   <!-- Little -->
-  <xacro:property name="little_proximal_length" value="0.025" />
-  <xacro:property name="little_proximal_width" value="0.015" />
-  <xacro:property name="little_proximal_depth" value="0.012" />
   <link name="little_proximal_link">
     <visual>
@@ -167,7 +145,4 @@
     </xacro:inertial_box>
   </link>
-  <xacro:property name="little_middle_length" value="0.05" />
-  <xacro:property name="little_middle_width" value="0.015" />
-  <xacro:property name="little_middle_depth" value="0.012" />
   <link name="little_middle_link">
     <visual>
@@ -184,7 +159,4 @@
   </link>
   <!-- Thumb -->
-  <xacro:property name="thumb_metacarpal_length" value="0.028" />
-  <xacro:property name="thumb_metacarpal_width" value="0.015" />
-  <xacro:property name="thumb_metacarpal_depth" value="0.012" />
   <link name="thumb_metacarpal_link">
     <visual>
@@ -200,7 +172,4 @@
     </xacro:inertial_box>
   </link>
-  <xacro:property name="thumb_proximal_length" value="0.025" />
-  <xacro:property name="thumb_proximal_width" value="0.015" />
-  <xacro:property name="thumb_proximal_depth" value="0.012" />
   <link name="thumb_proximal_link">
     <visual>
@@ -216,7 +185,4 @@
     </xacro:inertial_box>
   </link>
-  <xacro:property name="thumb_distal_length" value="0.020" />
-  <xacro:property name="thumb_distal_width" value="0.015" />
-  <xacro:property name="thumb_distal_depth" value="0.012" />
   <link name="thumb_distal_link">
     <visual>
@@ -253,13 +219,4 @@
     <limit lower="-1.57" upper="1.57" effort="5" velocity="5"/>
   </joint>
-  <!-- MCP X and Y positions for each finger relative to palm_link -->
-  <xacro:property name="mcp_x" value="${palm_length}" />
-  <xacro:property name="finger_width" value="${index_proximal_length}" />
-  <xacro:property name="spacing_area" value="${palm_width - finger_width * 4}"/>
-  <xacro:property name="d" value="${spacing_area / 5}"/>
-  <xacro:property name="index_mcp_y" value="${-palm_width / 2 + d + finger_width / 2}" />
-  <xacro:property name="middle_mcp_y" value="${-palm_width / 2 + d*2 + finger_width*1.5}" />
-  <xacro:property name="ring_mcp_y" value="${-palm_width / 2 + d*3 + finger_width*2.5}" />
-  <xacro:property name="little_mcp_y" value="${-palm_width / 2 + d*4 + finger_width*3.5}" />
   <!-- Index -->
   <joint name="joint_index_mcp" type="revolute">
@@ -309,5 +266,5 @@
   <joint name="joint_thumb_cmc" type="revolute">
     <parent link="palm_link"/><child link="thumb_metacarpal_link"/>
-    <origin xyz="${thumb_metacarpal_width/2} ${-(palm_width/2.5)} 0.00" rpy="0 0 -0.70"/><axis xyz="0 1 0"/>
+    <origin xyz="${thumb_metacarpal_width/2 + 0.02} ${-(palm_width/2) - 0.0068} 0.00" rpy="0 0 -0.80"/><axis xyz="0 1 0"/>
     <limit lower="-0.40" upper="1.20" effort="3" velocity="5"/>
   </joint>

Commit message: .  Changed base origin values for better accuracy in prosthesis.urdf.xacro .  Modified movement_input.py so the movement of grasping is decomposed in 3 different goals with timelaps . Deleted static property of the cylinder in prosthesis_world.sdf to it is subject to gravity

File: ros2_ws/src/prosthesis_description/model/prosthesis.urdf.xacro (robot description, xacro)
@@ -8,13 +8,13 @@
   <link name="base_link">
     <visual>
-        <origin xyz="${base_length/2} 0 0" rpy="0 0 0"/>
+        <origin xyz="${base_length/2} 0 ${base_depth/2}" rpy="0 0 0"/>
         <geometry><box size="${base_length} ${base_width} ${base_depth}"/></geometry>
     </visual>
     <collision>
-        <origin xyz="${base_length/2} 0 0" rpy="0 0 0"/>
+        <origin xyz="${base_length/2} 0 ${base_depth/2}" rpy="0 0 0"/>
         <geometry><box size="${base_length} ${base_width} ${base_depth}"/></geometry>
     </collision>
     <xacro:inertial_box mass="1.0" x="${base_length}" y="${base_width}" z="${base_depth}">
-        <origin xyz="${base_length/2} 0 0" rpy="0 0 0"/>
+        <origin xyz="${base_length/2} 0 ${base_depth/2}" rpy="0 0 0"/>
     </xacro:inertial_box>
   </link>
@@ -66,5 +66,5 @@
         <geometry><box size="${index_middle_length} ${index_middle_width} ${index_middle_depth}"/></geometry>
     </visual>
-    <collision>
+    <collision name="collision_index_middle">
         <origin xyz="${index_middle_length/2} 0 0" rpy="0 0 0"/>
         <geometry><box size="${index_middle_length} ${index_middle_width} ${index_middle_depth}"/></geometry>
@@ -109,5 +109,5 @@
         <geometry><box size="${middle_middle_length} ${middle_middle_width} ${middle_middle_depth}"/></geometry>
     </visual>
-    <collision>
+    <collision name="collision_middle_middle">
         <origin xyz="${middle_middle_length/2} 0 0" rpy="0 0 0"/>
         <geometry><box size="${middle_middle_length} ${middle_middle_width} ${middle_middle_depth}"/></geometry>
@@ -136,5 +136,5 @@
         <geometry><box size="${ring_middle_length} ${ring_middle_width} ${ring_middle_depth}"/></geometry>
     </visual>
-    <collision>
+    <collision name="collision_ring_middle">
         <origin xyz="${ring_middle_length/2} 0 0" rpy="0 0 0"/>
         <geometry><box size="${ring_middle_length} ${ring_middle_width} ${ring_middle_depth}"/></geometry>
@@ -163,5 +163,5 @@
         <geometry><box size="${little_middle_length} ${little_middle_width} ${little_middle_depth}"/></geometry>
     </visual>
-    <collision>
+    <collision name="collision_little_middle">
         <origin xyz="${little_middle_length/2} 0 0" rpy="0 0 0"/>
         <geometry><box size="${little_middle_length} ${little_middle_width} ${little_middle_depth}"/></geometry>
@@ -203,5 +203,5 @@
         <geometry><box size="${thumb_distal_length} ${thumb_distal_width} ${thumb_distal_depth}"/></geometry>
     </visual>
-    <collision>
+    <collision name="collision_thumb_distal">
         <origin xyz="${thumb_distal_length/2} 0 0" rpy="0 0 0"/>
         <geometry><box size="${thumb_distal_length} ${thumb_distal_width} ${thumb_distal_depth}"/></geometry>
@@ -222,5 +222,5 @@
     <parent link="base_link"/>
     <child  link="wrist_link"/>
-    <origin xyz="${base_length} 0 0" rpy="0 0 0"/>
+    <origin xyz="${base_length} 0 ${base_depth/2}" rpy="0 0 0"/>
   </joint>
   <!-- Wrist → Palm -->
@@ -229,5 +229,6 @@
     <child  link="palm_link"/>
     <origin xyz="${wrist_radius*2} 0 0" rpy="0 0 0"/>
-    <axis xyz="0 1 0"/>
+    <axis xyz="1 0 0"/>
+    <axis xyz="0 0 1"/>
     <limit lower="-1.57" upper="1.57" effort="5" velocity="5"/>
   </joint>

Commit message: Integrated first STL -- not to scale

File: ros2_ws/src/prosthesis_description/model/prosthesis.urdf.xacro (robot description, xacro)
@@ -23,5 +23,7 @@
       <visual>
           <origin xyz="0 0 0" rpy="0 0 0"/>
-          <geometry><box size="${base_length} ${base_width} ${base_depth}"/></geometry>
+          <geometry>
+            <mesh filename="$(find prosthesis_description)/meshes/PhalangeConstructrion_Base.stl" />
+          </geometry>
       </visual>
       <collision>

Commit message: Changed message type for arm mouvement goals and added links to urdf for roll pitch yaw mouvements of base arm

File: ros2_ws/src/prosthesis_description/model/prosthesis.urdf.xacro (robot description, xacro)
@@ -33,4 +33,22 @@
       </xacro:inertial_box>
     </link>
+    <link name="link_base_roll">
+      <inertial>
+        <mass value="0.001"/>
+        <inertia ixx="0.0001" ixy="0.0" ixz="0.0" iyy="0.0001" iyz="0.0" izz="0.0001"/>
+      </inertial>
+    </link>
+    <link name="link_base_pitch">
+      <inertial>
+        <mass value="0.001"/>
+        <inertia ixx="0.0001" ixy="0.0" ixz="0.0" iyy="0.0001" iyz="0.0" izz="0.0001"/>
+      </inertial>
+    </link>
+    <link name="link_base_yaw">
+      <inertial>
+        <mass value="0.001"/>
+        <inertia ixx="0.0001" ixy="0.0" ixz="0.0" iyy="0.0001" iyz="0.0" izz="0.0001"/>
+      </inertial>
+    </link>
     <xacro:property name="wrist_radius" value="0.01" />
     <link name="link_wrist_x">
@@ -326,5 +344,5 @@
           <child link="link_base_x"/>
           <axis xyz="1 0 0"/>
-          <limit lower="-1000" upper="1000" effort="100" velocity="1.0"/>
+          <limit lower="-1000" upper="1000" effort="100" velocity="4"/>
     </joint>
     <!-- Base X → Base Y (prismatic joint for y-axis motion) -->
@@ -334,5 +352,5 @@
           <child link="link_base_y"/>
           <axis xyz="0 1 0"/>
-          <limit lower="-1000" upper="1000" effort="100" velocity="1.0"/>
+          <limit lower="-1000" upper="1000" effort="100" velocity="4"/>
     </joint>
     <!-- Base Y → Base Link (prismatic joint for z-axis motion) -->
@@ -342,9 +360,33 @@
           <child link="link_base_z"/>
           <axis xyz="0 0 1"/>
-          <limit lower="0.0" upper="1000" effort="100" velocity="1.0"/>
+          <limit lower="-1000" upper="1000" effort="100" velocity="4"/>
+    </joint>
+    <!-- Base R → Base Link (revolute joint for roll motion) -->
+    <joint name="joint_base_roll" type="revolute">
+          <origin xyz="0 0 0" rpy="0 0 0"/>
+          <parent link="link_base_z"/>
+          <child link="link_base_roll"/>
+          <axis xyz="1 0 0"/>
+          <limit lower="-1.57" upper="1.57" effort="100" velocity="4"/>
+    </joint>
+    <!-- Base P → Base Link (revolute joint for pitch motion) -->
+    <joint name="joint_base_pitch" type="revolute">
+          <origin xyz="0 0 0" rpy="0 0 0"/>
+          <parent link="link_base_roll"/>
+          <child link="link_base_pitch"/>
+          <axis xyz="0 1 0"/>
+          <limit lower="-1.57" upper="1.57" effort="100" velocity="4"/>
+    </joint>
+    <!-- Base Y → Base Link (revolute joint for yaw motion) -->
+    <joint name="joint_base_yaw" type="revolute">
+          <origin xyz="0 0 0" rpy="0 0 0"/>
+          <parent link="link_base_pitch"/>
+          <child link="link_base_yaw"/>
+          <axis xyz="0 0 1"/>
+          <limit lower="-1.57" upper="1.57" effort="100" velocity="4"/>
     </joint>
     <!-- Base → Wrist -->
     <joint name="joint_base_to_wrist" type="fixed">
-      <parent link="link_base_z"/>
+      <parent link="link_base_yaw"/>
       <child  link="link_wrist_x"/>
       <origin xyz="0 0 ${wrist_radius}" rpy="0 0 0"/>
@@ -474,5 +516,5 @@
       <plugin>gz_ros2_control/GazeboSimSystem</plugin>
     </hardware>
-    <!-- Base Movement Joints (X, Y, Z) -->
+    <!-- Base Movement Joints (x, y, z, r, p, y) -->
     <joint name="joint_base_x">
       <command_interface name="position"/> <!-- command controller will send for position control -->
@@ -493,4 +535,22 @@
       <state_interface name="effort"/>
     </joint>
+    <joint name="joint_base_roll">
+      <command_interface name="position"/>
+      <state_interface name="position"/>
+      <state_interface name="velocity"/>
+      <state_interface name="effort"/>
+    </joint>
+    <joint name="joint_base_pitch">
+      <command_interface name="position"/>
+      <state_interface name="position"/>
+      <state_interface name="velocity"/>
+      <state_interface name="effort"/>
+    </joint>
+    <joint name="joint_base_yaw">
+      <command_interface name="position"/>
+      <state_interface name="position"/>
+      <state_interface name="velocity"/>
+      <state_interface name="effort"/>
+    </joint>
     <!-- Wrist Joint -->
     <joint name="joint_wrist_x">
