Commit message: changes for ros2 control integration (#2)

File: ros2_ws/src/prosthesis_description/model/gazebo.xacro (robot description, xacro)
@@ -84,11 +84,5 @@
     </joint>
   </ros2_control>
-    <!-- ===== GAZEBO TAGS ===== -->
-  <xacro:property name="base_wrist_friction" value="0.8" />
-  <xacro:property name="palm_fingers_friction" value="1" />
-  <xacro:property name="rigid_stiffness_default" value="1000000" />
-  <xacro:property name="damping_default" value="200" /> <!-- contact damping prevents bouncing and oscillation. kd is approximately 2*sqrt(kp*m) -->
-  <xacro:property name="min_depth_default" value="0.001" />
-  <xacro:property name="max_velocity_default" value="1" />
+  <!-- ===== GAZEBO TAGS ===== -->
   <!-- Base and palm Gazebo tags -->
   <gazebo reference="base_link">
@@ -97,5 +91,5 @@
     <mu2>${base_wrist_friction}</mu2>
     <kp>${rigid_stiffness_default}</kp> <!-- Contact stiffness -->
-    <kd>${damping_default}</kd> <!-- Contact damping (prevents bounce)-->
+    <kd>${damping_default}</kd> <!-- Contact damping (prevents bounce, kd is approximately 2*sqrt(kp*m)-->
     <minDepth>${min_depth_default}</minDepth> <!-- Minimum depth for contact -->
     <maxVel>${max_velocity_default}</maxVel> <!-- Maximum velocity for contact -->

File: ros2_ws/src/prosthesis_description/model/prosthesis.urdf.xacro (robot description, xacro)
@@ -1,11 +1,8 @@
 <?xml version="1.0"?>
 <robot xmlns:xacro="http://www.ros.org/wiki/xacro" name="hand">
-<xacro:include filename="useful_tags.xacro" />
-<xacro:include filename="prosthesis.gazebo.urdf" />
+<xacro:include filename="parameters.xacro" />
+<xacro:include filename="gazebo.xacro" />
   <!-- ===== LINKS (base & palm unchanged) ===== -->
   <link name="world" />
-  <xacro:property name="base_length" value="0.174" />
-  <xacro:property name="base_width" value="0.065" />
-  <xacro:property name="base_depth" value="0.101" />
   <link name="base_link">
     <visual>
@@ -35,7 +32,4 @@
     </xacro:inertial_sphere>
   </link>
-  <xacro:property name="palm_length" value="0.068" />
-  <xacro:property name="palm_width" value="0.098" />
-  <xacro:property name="palm_depth" value="0.019" />
   <link name="palm_link">
     <visual>
@@ -53,7 +47,4 @@
   <!-- ===== FINGER & THUMB LINKS (all boxes 0.02 x 0.05 x 0.02) ===== -->
   <!-- Index -->
-  <xacro:property name="index_proximal_length" value="0.025" />
-  <xacro:property name="index_proximal_width" value="0.015" />
-  <xacro:property name="index_proximal_depth" value="0.012" />
   <link name="index_proximal_link">
     <visual>
@@ -69,7 +60,4 @@
     </xacro:inertial_box>
   </link>
-  <xacro:property name="index_middle_length" value="0.05" />
-  <xacro:property name="index_middle_width" value="0.015" />
-  <xacro:property name="index_middle_depth" value="0.012" />
   <link name="index_middle_link">
     <visual>
@@ -86,7 +74,4 @@
   </link>
   <!-- Middle -->
-  <xacro:property name="middle_proximal_length" value="0.025" />
-  <xacro:property name="middle_proximal_width" value="0.015" />
-  <xacro:property name="middle_proximal_depth" value="0.012" />
   <link name="middle_proximal_link">
     <visual>
@@ -119,7 +104,4 @@
   </link>
   <!-- Ring -->
-  <xacro:property name="ring_proximal_length" value="0.025" />
-  <xacro:property name="ring_proximal_width" value="0.015" />
-  <xacro:property name="ring_proximal_depth" value="0.012" />
   <link name="ring_proximal_link">
     <visual>
@@ -135,7 +117,4 @@
     </xacro:inertial_box>
   </link>
-  <xacro:property name="ring_middle_length" value="0.05" />
-  <xacro:property name="ring_middle_width" value="0.015" />
-  <xacro:property name="ring_middle_depth" value="0.012" />
   <link name="ring_middle_link">
     <visual>
@@ -152,7 +131,4 @@
   </link>
   <!-- Little -->
-  <xacro:property name="little_proximal_length" value="0.025" />
-  <xacro:property name="little_proximal_width" value="0.015" />
-  <xacro:property name="little_proximal_depth" value="0.012" />
   <link name="little_proximal_link">
     <visual>
@@ -168,7 +144,4 @@
     </xacro:inertial_box>
   </link>
-  <xacro:property name="little_middle_length" value="0.05" />
-  <xacro:property name="little_middle_width" value="0.015" />
-  <xacro:property name="little_middle_depth" value="0.012" />
   <link name="little_middle_link">
     <visual>
@@ -185,7 +158,4 @@
   </link>
   <!-- Thumb -->
-  <xacro:property name="thumb_metacarpal_length" value="0.028" />
-  <xacro:property name="thumb_metacarpal_width" value="0.015" />
-  <xacro:property name="thumb_metacarpal_depth" value="0.012" />
   <link name="thumb_metacarpal_link">
     <visual>
@@ -201,7 +171,4 @@
     </xacro:inertial_box>
   </link>
-  <xacro:property name="thumb_proximal_length" value="0.025" />
-  <xacro:property name="thumb_proximal_width" value="0.015" />
-  <xacro:property name="thumb_proximal_depth" value="0.012" />
   <link name="thumb_proximal_link">
     <visual>
@@ -217,7 +184,4 @@
     </xacro:inertial_box>
   </link>
-  <xacro:property name="thumb_distal_length" value="0.020" />
-  <xacro:property name="thumb_distal_width" value="0.015" />
-  <xacro:property name="thumb_distal_depth" value="0.012" />
   <link name="thumb_distal_link">
     <visual>
@@ -254,13 +218,4 @@
     <limit lower="-1.57" upper="1.57" effort="5" velocity="5"/>
   </joint>
-  <!-- MCP X and Y positions for each finger relative to palm_link -->
-  <xacro:property name="mcp_x" value="${palm_length}" />
-  <xacro:property name="finger_width" value="${index_proximal_length}" />
-  <xacro:property name="spacing_area" value="${palm_width - finger_width * 4}"/>
-  <xacro:property name="d" value="${spacing_area / 5}"/>
-  <xacro:property name="index_mcp_y" value="${-palm_width / 2 + d + finger_width / 2}" />
-  <xacro:property name="middle_mcp_y" value="${-palm_width / 2 + d*2 + finger_width*1.5}" />
-  <xacro:property name="ring_mcp_y" value="${-palm_width / 2 + d*3 + finger_width*2.5}" />
-  <xacro:property name="little_mcp_y" value="${-palm_width / 2 + d*4 + finger_width*3.5}" />
   <!-- Index -->
   <joint name="joint_index_mcp" type="revolute">

Commit message: Working basic gz_ros2_control plugin

File: ros2_ws/src/prosthesis_description/model/gazebo.xacro (robot description, xacro)
@@ -1,4 +1,137 @@
 <?xml version="1.0"?>
 <robot xmlns:xacro="http://www.ros.org/wiki/xacro">
+<!-- File containing all additional descriptions necessary for Gazebo simulation-->
+  <!-- ===== GAZEBO TAGS ===== -->
+  <!-- Needed additional link properties to simulate robot in accurate physics environment-->
+  <!-- Base and palm Gazebo tags -->
+  <gazebo reference="base_link">
+    <material>Gazebo/Gray</material> <!-- Visual material used in Gazebo GUI -->
+    <mu1>${base_wrist_friction}</mu1> <!-- Friction coefficients -->
+    <mu2>${base_wrist_friction}</mu2>
+    <kp>${rigid_stiffness_default}</kp> <!-- Contact stiffness -->
+    <kd>${damping_default}</kd> <!-- Contact damping (prevents bounce, kd is approximately 2*sqrt(kp*m)-->
+    <minDepth>${min_depth_default}</minDepth> <!-- Minimum depth for contact -->
+    <maxVel>${max_velocity_default}</maxVel> <!-- Maximum velocity for contact -->
+  </gazebo>
+  <gazebo reference="wrist_link">
+    <material>Gazebo/White</material>
+    <mu1>${base_wrist_friction}</mu1>
+    <mu2>${base_wrist_friction}</mu2>
+    <kp>${rigid_stiffness_default}</kp>
+    <kd>${damping_default}</kd>
+    <minDepth>${min_depth_default}</minDepth>
+  </gazebo>
+  <gazebo reference="palm_link">
+    <material>Gazebo/Orange</material>
+    <mu1>${palm_fingers_friction}</mu1>
+    <mu2>${palm_fingers_friction}</mu2>
+    <kp>${rigid_stiffness_default}</kp>
+    <kd>${damping_default}</kd>
+    <minDepth>${min_depth_default}</minDepth>
+  </gazebo>
+  <!-- Index finger Gazebo tags -->
+  <gazebo reference="index_proximal_link">
+    <material>Gazebo/SkyBlue</material>
+    <mu1>${palm_fingers_friction}</mu1>
+    <mu2>${palm_fingers_friction}</mu2>
+    <kp>${rigid_stiffness_default}</kp>
+    <kd>${damping_default}</kd>
+    <minDepth>${min_depth_default}</minDepth>
+    <maxVel>${max_velocity_default}</maxVel>
+  </gazebo>
+  <gazebo reference="index_middle_link">
+    <material>Gazebo/Blue</material>
+    <mu1>${palm_fingers_friction}</mu1>
+    <mu2>${palm_fingers_friction}</mu2>
+    <kp>${rigid_stiffness_default}</kp>
+    <kd>${damping_default}</kd>
+    <minDepth>${min_depth_default}</minDepth>
+    <maxVel>${max_velocity_default}</maxVel>
+  </gazebo>
+  <!-- Middle finger Gazebo tags -->
+  <gazebo reference="middle_proximal_link">
+    <material>Gazebo/SkyBlue</material>
+    <mu1>${palm_fingers_friction}</mu1>
+    <mu2>${palm_fingers_friction}</mu2>
+    <kp>${rigid_stiffness_default}</kp>
+    <kd>${damping_default}</kd>
+    <minDepth>${min_depth_default}</minDepth>
+    <maxVel>${max_velocity_default}</maxVel>
+  </gazebo>
+  <gazebo reference="middle_middle_link">
+    <material>Gazebo/Blue</material>
+    <mu1>${palm_fingers_friction}</mu1>
+    <mu2>${palm_fingers_friction}</mu2>
+    <kp>${rigid_stiffness_default}</kp>
+    <kd>${damping_default}</kd>
+    <minDepth>${min_depth_default}</minDepth>
+    <maxVel>${max_velocity_default}</maxVel>
+  </gazebo>
+  <!-- Ring finger Gazebo tags -->
+  <gazebo reference="ring_proximal_link">
+    <material>Gazebo/SkyBlue</material>
+    <mu1>${palm_fingers_friction}</mu1>
+    <mu2>${palm_fingers_friction}</mu2>
+    <kp>${rigid_stiffness_default}</kp>
+    <kd>${damping_default}</kd>
+    <minDepth>${min_depth_default}</minDepth>
+    <maxVel>${max_velocity_default}</maxVel>
+  </gazebo>
+  <gazebo reference="ring_middle_link">
+    <material>Gazebo/Blue</material>
+    <mu1>${palm_fingers_friction}</mu1>
+    <mu2>${palm_fingers_friction}</mu2>
+    <kp>${rigid_stiffness_default}</kp>
+    <kd>${damping_default}</kd>
+    <minDepth>${min_depth_default}</minDepth>
+    <maxVel>${max_velocity_default}</maxVel>
+  </gazebo>
+  <!-- Little finger Gazebo tags -->
+  <gazebo reference="little_proximal_link">
+    <material>Gazebo/SkyBlue</material>
+    <mu1>${palm_fingers_friction}</mu1>
+    <mu2>${palm_fingers_friction}</mu2>
+    <kp>${rigid_stiffness_default}</kp>
+    <kd>${damping_default}</kd>
+    <minDepth>${min_depth_default}</minDepth>
+    <maxVel>${max_velocity_default}</maxVel>
+  </gazebo>
+  <gazebo reference="little_middle_link">
+    <material>Gazebo/Blue</material>
+    <mu1>${palm_fingers_friction}</mu1>
+    <mu2>${palm_fingers_friction}</mu2>
+    <kp>${rigid_stiffness_default}</kp>
+    <kd>${damping_default}</kd>
+    <minDepth>${min_depth_default}</minDepth>
+    <maxVel>${max_velocity_default}</maxVel>
+  </gazebo>
+  <!-- Thumb Gazebo tags -->
+  <gazebo reference="thumb_metacarpal_link">
+    <material>Gazebo/Green</material>
+    <mu1>${palm_fingers_friction}</mu1>
+    <mu2>${palm_fingers_friction}</mu2>
+    <kp>${rigid_stiffness_default}</kp>
+    <kd>${damping_default}</kd>
+    <minDepth>${min_depth_default}</minDepth>
+    <maxVel>${max_velocity_default}</maxVel>
+  </gazebo>
+  <gazebo reference="thumb_proximal_link">
+    <material>Gazebo/Green</material>
+    <mu1>${palm_fingers_friction}</mu1>
+    <mu2>${palm_fingers_friction}</mu2>
+    <kp>${rigid_stiffness_default}</kp>
+    <kd>${damping_default}</kd>
+    <minDepth>${min_depth_default}</minDepth>
+    <maxVel>${max_velocity_default}</maxVel>
+  </gazebo>
+  <gazebo reference="thumb_distal_link">
+    <material>Gazebo/Green</material>
+    <mu1>${palm_fingers_friction}</mu1>
+    <mu2>${palm_fingers_friction}</mu2>
+    <kp>${rigid_stiffness_default}</kp>
+    <kd>${damping_default}</kd>
+    <minDepth>${min_depth_default}</minDepth>
+    <maxVel>${max_velocity_default}</maxVel>
+  </gazebo>
   <!-- ===== GAZEBO ROS2 CONTROL PLUGIN ===== -->
   <!-- Bridges Gazebo simulation to ROS2 controller manager
@@ -8,4 +141,5 @@
     <plugin filename="gz_ros2_control-system" name="gz_ros2_control::GazeboSimROS2ControlPlugin">
       <parameters>$(find prosthesis_description)/config/prosthesis_controllers.yaml</parameters>
+      <controller_manager_prefix_node_name>controller_manager</controller_manager_prefix_node_name>
     </plugin>
   </gazebo>
@@ -84,134 +218,3 @@
     </joint>
   </ros2_control>
-  <!-- ===== GAZEBO TAGS ===== -->
-  <!-- Base and palm Gazebo tags -->
-  <gazebo reference="base_link">
-    <material>Gazebo/Gray</material> <!-- Visual material used in Gazebo GUI -->
-    <mu1>${base_wrist_friction}</mu1> <!-- Friction coefficients -->
-    <mu2>${base_wrist_friction}</mu2>
-    <kp>${rigid_stiffness_default}</kp> <!-- Contact stiffness -->
-    <kd>${damping_default}</kd> <!-- Contact damping (prevents bounce, kd is approximately 2*sqrt(kp*m)-->
-    <minDepth>${min_depth_default}</minDepth> <!-- Minimum depth for contact -->
-    <maxVel>${max_velocity_default}</maxVel> <!-- Maximum velocity for contact -->
-  </gazebo>
-  <gazebo reference="wrist_link">
-    <material>Gazebo/White</material>
-    <mu1>${base_wrist_friction}</mu1>
-    <mu2>${base_wrist_friction}</mu2>
-    <kp>${rigid_stiffness_default}</kp>
-    <kd>${damping_default}</kd>
-    <minDepth>${min_depth_default}</minDepth>
-  </gazebo>
-  <gazebo reference="palm_link">
-    <material>Gazebo/Orange</material>
-    <mu1>${palm_fingers_friction}</mu1>
-    <mu2>${palm_fingers_friction}</mu2>
-    <kp>${rigid_stiffness_default}</kp>
-    <kd>${damping_default}</kd>
-    <minDepth>${min_depth_default}</minDepth>
-  </gazebo>
-  <!-- Index finger Gazebo tags -->
-  <gazebo reference="index_proximal_link">
-    <material>Gazebo/SkyBlue</material>
-    <mu1>${palm_fingers_friction}</mu1>
-    <mu2>${palm_fingers_friction}</mu2>
-    <kp>${rigid_stiffness_default}</kp>
-    <kd>${damping_default}</kd>
-    <minDepth>${min_depth_default}</minDepth>
-    <maxVel>${max_velocity_default}</maxVel>
-  </gazebo>
-  <gazebo reference="index_middle_link">
-    <material>Gazebo/Blue</material>
-    <mu1>${palm_fingers_friction}</mu1>
-    <mu2>${palm_fingers_friction}</mu2>
-    <kp>${rigid_stiffness_default}</kp>
-    <kd>${damping_default}</kd>
-    <minDepth>${min_depth_default}</minDepth>
-    <maxVel>${max_velocity_default}</maxVel>
-  </gazebo>
-  <!-- Middle finger Gazebo tags -->
-  <gazebo reference="middle_proximal_link">
-    <material>Gazebo/SkyBlue</material>
-    <mu1>${palm_fingers_friction}</mu1>
-    <mu2>${palm_fingers_friction}</mu2>
-    <kp>${rigid_stiffness_default}</kp>
-    <kd>${damping_default}</kd>
-    <minDepth>${min_depth_default}</minDepth>
-    <maxVel>${max_velocity_default}</maxVel>
-  </gazebo>
-  <gazebo reference="middle_middle_link">
-    <material>Gazebo/Blue</material>
-    <mu1>${palm_fingers_friction}</mu1>
-    <mu2>${palm_fingers_friction}</mu2>
-    <kp>${rigid_stiffness_default}</kp>
-    <kd>${damping_default}</kd>
-    <minDepth>${min_depth_default}</minDepth>
-    <maxVel>${max_velocity_default}</maxVel>
-  </gazebo>
-  <!-- Ring finger Gazebo tags -->
-  <gazebo reference="ring_proximal_link">
-    <material>Gazebo/SkyBlue</material>
-    <mu1>${palm_fingers_friction}</mu1>
-    <mu2>${palm_fingers_friction}</mu2>
-    <kp>${rigid_stiffness_default}</kp>
-    <kd>${damping_default}</kd>
-    <minDepth>${min_depth_default}</minDepth>
-    <maxVel>${max_velocity_default}</maxVel>
-  </gazebo>
-  <gazebo reference="ring_middle_link">
-    <material>Gazebo/Blue</material>
-    <mu1>${palm_fingers_friction}</mu1>
-    <mu2>${palm_fingers_friction}</mu2>
-    <kp>${rigid_stiffness_default}</kp>
-    <kd>${damping_default}</kd>
-    <minDepth>${min_depth_default}</minDepth>
-    <maxVel>${max_velocity_default}</maxVel>
-  </gazebo>
-  <!-- Little finger Gazebo tags -->
-  <gazebo reference="little_proximal_link">
-    <material>Gazebo/SkyBlue</material>
-    <mu1>${palm_fingers_friction}</mu1>
-    <mu2>${palm_fingers_friction}</mu2>
-    <kp>${rigid_stiffness_default}</kp>
-    <kd>${damping_default}</kd>
-    <minDepth>${min_depth_default}</minDepth>
-    <maxVel>${max_velocity_default}</maxVel>
-  </gazebo>
-  <gazebo reference="little_middle_link">
-    <material>Gazebo/Blue</material>
-    <mu1>${palm_fingers_friction}</mu1>
-    <mu2>${palm_fingers_friction}</mu2>
-    <kp>${rigid_stiffness_default}</kp>
-    <kd>${damping_default}</kd>
-    <minDepth>${min_depth_default}</minDepth>
-    <maxVel>${max_velocity_default}</maxVel>
-  </gazebo>
-  <!-- Thumb Gazebo tags -->
-  <gazebo reference="thumb_metacarpal_link">
-    <material>Gazebo/Green</material>
-    <mu1>${palm_fingers_friction}</mu1>
-    <mu2>${palm_fingers_friction}</mu2>
-    <kp>${rigid_stiffness_default}</kp>
-    <kd>${damping_default}</kd>
-    <minDepth>${min_depth_default}</minDepth>
-    <maxVel>${max_velocity_default}</maxVel>
-  </gazebo>
-  <gazebo reference="thumb_proximal_link">
-    <material>Gazebo/Green</material>
-    <mu1>${palm_fingers_friction}</mu1>
-    <mu2>${palm_fingers_friction}</mu2>
-    <kp>${rigid_stiffness_default}</kp>
-    <kd>${damping_default}</kd>
-    <minDepth>${min_depth_default}</minDepth>
-    <maxVel>${max_velocity_default}</maxVel>
-  </gazebo>
-  <gazebo reference="thumb_distal_link">
-    <material>Gazebo/Green</material>
-    <mu1>${palm_fingers_friction}</mu1>
-    <mu2>${palm_fingers_friction}</mu2>
-    <kp>${rigid_stiffness_default}</kp>
-    <kd>${damping_default}</kd>
-    <minDepth>${min_depth_default}</minDepth>
-    <maxVel>${max_velocity_default}</maxVel>
-  </gazebo>
 </robot>

File: ros2_ws/src/prosthesis_description/model/parameters.xacro (robot description, xacro)
@@ -1,4 +1,5 @@
 <?xml version="1.0"?>
 <robot xmlns:xacro="http://www.ros.org/wiki/xacro" >
+<!-- File containing all useful values for the robot description -->
     <!-- ==== PROSTHESIS VALUES ==== -->
     <!-- Dimensions for each link -->

File: ros2_ws/src/prosthesis_description/model/prosthesis.urdf.xacro (robot description, xacro)
@@ -1,4 +1,5 @@
 <?xml version="1.0"?>
 <robot xmlns:xacro="http://www.ros.org/wiki/xacro" name="hand">
+<!--File containing all the fundamental links and joints description-->
 <xacro:include filename="parameters.xacro" />
 <xacro:include filename="gazebo.xacro" />

Commit message: - added object to world - tried to add sensors to finger's last links but problem with gz-ros bridging - fsr_broadcaster.py node subscribes to contact topic from Gazebo and adds Gaussian noise and normalizes value -joint_state_printer also prints the fsr like value

File: ros2_ws/src/prosthesis_description/model/gazebo.xacro (robot description, xacro)
@@ -2,6 +2,15 @@
 <robot xmlns:xacro="http://www.ros.org/wiki/xacro">
 <!-- File containing all additional descriptions necessary for Gazebo simulation-->
-  <!-- ===== GAZEBO TAGS ===== -->
+  <!-- ===== GAZEBO TAGS ROS2 CONTROL PLUGIN ===== -->
   <!-- Needed additional link properties to simulate robot in accurate physics environment-->
+  <!-- Plugin bridges Gazebo simulation to ROS2 controller manager
+  by reading YAML config file (update rates, controllers to load, namespaces)
+  and initializes hardware interface which exposes joint read/write methods to ros2_control -->
+  <gazebo>
+    <plugin filename="gz_ros2_control-system" name="gz_ros2_control::GazeboSimROS2ControlPlugin">
+      <parameters>$(find prosthesis_description)/config/prosthesis_controllers.yaml</parameters>
+      <controller_manager_prefix_node_name>controller_manager</controller_manager_prefix_node_name>
+    </plugin>
+  </gazebo>
   <!-- Base and palm Gazebo tags -->
   <gazebo reference="base_link">
@@ -48,4 +57,11 @@
     <minDepth>${min_depth_default}</minDepth>
     <maxVel>${max_velocity_default}</maxVel>
+    <sensor name="index_fsr" type="contact">
+      <always_on>true</always_on>
+      <update_rate>1000</update_rate>
+      <contact>
+        <collision>collision</collision>
+      </contact>
+    </sensor>
   </gazebo>
   <!-- Middle finger Gazebo tags -->
@@ -67,4 +83,11 @@
     <minDepth>${min_depth_default}</minDepth>
     <maxVel>${max_velocity_default}</maxVel>
+    <sensor name="middle_fsr" type="contact">
+      <always_on>true</always_on>
+      <update_rate>1000</update_rate>
+      <contact>
+        <collision>collision</collision>
+      </contact>
+    </sensor>
   </gazebo>
   <!-- Ring finger Gazebo tags -->
@@ -86,4 +109,11 @@
     <minDepth>${min_depth_default}</minDepth>
     <maxVel>${max_velocity_default}</maxVel>
+    <sensor name="ring_fsr" type="contact">
+      <always_on>true</always_on>
+      <update_rate>1000</update_rate>
+      <contact>
+        <collision>collision</collision>
+      </contact>
+    </sensor>
   </gazebo>
   <!-- Little finger Gazebo tags -->
@@ -105,4 +135,11 @@
     <minDepth>${min_depth_default}</minDepth>
     <maxVel>${max_velocity_default}</maxVel>
+    <sensor name="little_fsr" type="contact">
+      <always_on>true</always_on>
+      <update_rate>1000</update_rate>
+      <contact>
+        <collision>collision</collision>
+      </contact>
+    </sensor>
   </gazebo>
   <!-- Thumb Gazebo tags -->
@@ -133,14 +170,11 @@
     <minDepth>${min_depth_default}</minDepth>
     <maxVel>${max_velocity_default}</maxVel>
-  </gazebo>
-  <!-- ===== GAZEBO ROS2 CONTROL PLUGIN ===== -->
-  <!-- Bridges Gazebo simulation to ROS2 controller manager
-  by reading YAML config file (update rates, controllers to load, namespaces)
-  and initializes hardware interface which exposes joint read/write methods to ros2_control -->
-  <gazebo>
-    <plugin filename="gz_ros2_control-system" name="gz_ros2_control::GazeboSimROS2ControlPlugin">
-      <parameters>$(find prosthesis_description)/config/prosthesis_controllers.yaml</parameters>
-      <controller_manager_prefix_node_name>controller_manager</controller_manager_prefix_node_name>
-    </plugin>
+    <sensor name="thumb_fsr" type="contact">
+      <always_on>true</always_on>
+      <update_rate>1000</update_rate>
+      <contact>
+        <collision>collision</collision>
+      </contact>
+    </sensor>
   </gazebo>
   <!-- ===== ROS2 CONTROL INTERFACE ===== -->

File: ros2_ws/src/prosthesis_description/model/prosthesis.urdf.xacro (robot description, xacro)
@@ -201,5 +201,5 @@
   <!-- World → Base -->
   <joint name="joint_world_to_base" type="fixed">
-        <origin xyz="0 0 ${base_depth/2}" rpy="0 0 0"/>
+        <origin xyz="0 0 0" rpy="0 0 0"/>
         <parent link="world"/>
         <child link="base_link"/>
