Commit message: add IMU and change FSR (not working)

File: ros2_ws/src/prosthesis_description/model/gazebo.xacro (robot description, xacro)
@@ -57,11 +57,4 @@
     <minDepth>${min_depth_default}</minDepth>
     <maxVel>${max_velocity_default}</maxVel>
-    <sensor name="index_fsr" type="contact">
-      <always_on>true</always_on>
-      <update_rate>1000</update_rate>
-      <contact>
-        <collision>collision</collision>
-      </contact>
-    </sensor>
   </gazebo>
   <!-- Middle finger Gazebo tags -->
@@ -83,11 +76,4 @@
     <minDepth>${min_depth_default}</minDepth>
     <maxVel>${max_velocity_default}</maxVel>
-    <sensor name="middle_fsr" type="contact">
-      <always_on>true</always_on>
-      <update_rate>1000</update_rate>
-      <contact>
-        <collision>collision</collision>
-      </contact>
-    </sensor>
   </gazebo>
   <!-- Ring finger Gazebo tags -->
@@ -109,11 +95,4 @@
     <minDepth>${min_depth_default}</minDepth>
     <maxVel>${max_velocity_default}</maxVel>
-    <sensor name="ring_fsr" type="contact">
-      <always_on>true</always_on>
-      <update_rate>1000</update_rate>
-      <contact>
-        <collision>collision</collision>
-      </contact>
-    </sensor>
   </gazebo>
   <!-- Little finger Gazebo tags -->
@@ -135,11 +114,4 @@
     <minDepth>${min_depth_default}</minDepth>
     <maxVel>${max_velocity_default}</maxVel>
-    <sensor name="little_fsr" type="contact">
-      <always_on>true</always_on>
-      <update_rate>1000</update_rate>
-      <contact>
-        <collision>collision</collision>
-      </contact>
-    </sensor>
   </gazebo>
   <!-- Thumb Gazebo tags -->
@@ -170,4 +142,50 @@
     <minDepth>${min_depth_default}</minDepth>
     <maxVel>${max_velocity_default}</maxVel>
+  </gazebo>
+  <!-- IMU -->
+  <gazebo reference="palm_link">
+    <sensor name="imu_sensor" type="imu">
+      <always_on>true</always_on>
+      <update_rate>50</update_rate>
+    </sensor>
+  </gazebo>
+  <!-- FSR -->
+  <gazebo reference="index_middle_fsr_link">
+    <sensor name="index_fsr" type="contact">
+      <always_on>true</always_on>
+      <update_rate>1000</update_rate>
+      <contact>
+        <collision>collision</collision>
+      </contact>
+    </sensor>
+  </gazebo>
+  <gazebo reference="middle_middle_link">
+      <sensor name="middle_fsr" type="contact">
+      <always_on>true</always_on>
+      <update_rate>1000</update_rate>
+      <contact>
+        <collision>collision</collision>
+      </contact>
+    </sensor>
+  </gazebo>
+  <gazebo reference="ring_middle_link">
+    <sensor name="ring_fsr" type="contact">
+      <always_on>true</always_on>
+      <update_rate>1000</update_rate>
+      <contact>
+        <collision>collision</collision>
+      </contact>
+    </sensor>
+  </gazebo>
+  <gazebo reference="little_middle_link">
+    <sensor name="little_fsr" type="contact">
+      <always_on>true</always_on>
+      <update_rate>1000</update_rate>
+      <contact>
+        <collision>collision</collision>
+      </contact>
+    </sensor>
+  </gazebo>
+  <gazebo reference="thumb_distal_link">
     <sensor name="thumb_fsr" type="contact">
       <always_on>true</always_on>

File: ros2_ws/src/prosthesis_description/model/prosthesis.urdf.xacro (robot description, xacro)
@@ -69,4 +69,17 @@
         <origin xyz="${index_middle_length/2} 0 0" rpy="0 0 0"/>
         <geometry><box size="${index_middle_length} ${index_middle_width} ${index_middle_depth}"/></geometry>
+    </collision>
+    <xacro:inertial_box mass="0.02" x="${index_middle_length}" y="${index_middle_width}" z="${index_middle_depth}">
+        <origin xyz="${index_middle_length/2} 0 0" rpy="0 0 0"/>
+    </xacro:inertial_box>
+  </link>
+  <link name="index_middle_fsr_link">
+    <visual>
+        <origin xyz="${index_middle_length/2} 0 -0.005" rpy="0 0 0"/>
+        <geometry><sphere radius="0.005"/></geometry>
+    </visual>
+    <collision>
+        <origin xyz="${index_middle_length/2} 0 0" rpy="0 0 0"/>
+        <geometry><sphere radius="0.005"/></geometry>
     </collision>
     <xacro:inertial_box mass="0.02" x="${index_middle_length}" y="${index_middle_width}" z="${index_middle_depth}">
@@ -230,4 +243,8 @@
     <limit lower="0.0" upper="1.57" effort="2" velocity="5"/>
   </joint>
+  <joint name="joint_index_fsr" type="fixed">
+    <parent link="index_middle_link"/><child link="index_middle_fsr_link"/>
+    <origin xyz="${index_middle_length/2} 0 0" rpy="0 0 0"/>
+  </joint>
   <!-- Middle -->
   <joint name="joint_middle_mcp" type="revolute">

Commit message: . Added keyboard control for prosthesis arm (base) Had to decompose the base joint and links to be able to move the arm in x y and z direction . Deleted useless timerAction in gazebo.launch.py for spawning entity

File: ros2_ws/src/prosthesis_description/model/gazebo.xacro (robot description, xacro)
@@ -204,4 +204,20 @@
       <plugin>gz_ros2_control/GazeboSimSystem</plugin>
     </hardware>
+    <!-- Base Movement Joints (X, Y, Z) -->
+    <joint name="joint_world_to_base_x">
+      <command_interface name="position"/>
+      <state_interface name="position"/>
+      <state_interface name="velocity"/>
+    </joint>
+    <joint name="joint_base_x_to_base_y">
+      <command_interface name="position"/>
+      <state_interface name="position"/>
+      <state_interface name="velocity"/>
+    </joint>
+    <joint name="joint_base_y_to_base_z">
+      <command_interface name="position"/>
+      <state_interface name="position"/>
+      <state_interface name="velocity"/>
+    </joint>
     <!-- Wrist Joint -->
     <joint name="joint_wrist_to_palm">

File: ros2_ws/src/prosthesis_description/model/prosthesis.urdf.xacro (robot description, xacro)
@@ -6,15 +6,28 @@
   <!-- ===== LINKS (base & palm unchanged) ===== -->
   <link name="world" />
+  <!-- Intermediate kinematic links for base movement (x, y, z) -->
+  <link name="base_link_x_frame">
+    <inertial>
+      <mass value="0.001"/>
+      <inertia ixx="0.0001" ixy="0.0" ixz="0.0" iyy="0.0001" iyz="0.0" izz="0.0001"/>
+    </inertial>
+  </link>
+  <link name="base_link_y_frame">
+    <inertial>
+      <mass value="0.001"/>
+      <inertia ixx="0.0001" ixy="0.0" ixz="0.0" iyy="0.0001" iyz="0.0" izz="0.0001"/>
+    </inertial>
+  </link>
   <link name="base_link">
     <visual>
-        <origin xyz="${base_length/2} 0 ${base_depth/2}" rpy="0 0 0"/>
+        <origin xyz="0 0 0" rpy="0 0 0"/>
         <geometry><box size="${base_length} ${base_width} ${base_depth}"/></geometry>
     </visual>
     <collision>
-        <origin xyz="${base_length/2} 0 ${base_depth/2}" rpy="0 0 0"/>
+        <origin xyz="0 0 0" rpy="0 0 0"/>
         <geometry><box size="${base_length} ${base_width} ${base_depth}"/></geometry>
     </collision>
     <xacro:inertial_box mass="1.0" x="${base_length}" y="${base_width}" z="${base_depth}">
-        <origin xyz="${base_length/2} 0 ${base_depth/2}" rpy="0 0 0"/>
+        <origin xyz="0 0 0" rpy="0 0 0"/>
     </xacro:inertial_box>
   </link>
@@ -212,15 +225,33 @@
   </link>
   <!-- ===== JOINTS ===== -->
-  <!-- World → Base -->
-  <joint name="joint_world_to_base" type="fixed">
+  <!-- World → Base X (prismatic joint for x-axis motion) -->
+  <joint name="joint_world_to_base_x" type="prismatic">
         <origin xyz="0 0 0" rpy="0 0 0"/>
         <parent link="world"/>
+        <child link="base_link_x_frame"/>
+        <axis xyz="1 0 0"/>
+        <limit lower="-2.0" upper="2.0" effort="100" velocity="1.0"/>
+  </joint>
+  <!-- Base X → Base Y (prismatic joint for y-axis motion) -->
+  <joint name="joint_base_x_to_base_y" type="prismatic">
+        <origin xyz="0 0 0" rpy="0 0 0"/>
+        <parent link="base_link_x_frame"/>
+        <child link="base_link_y_frame"/>
+        <axis xyz="0 1 0"/>
+        <limit lower="-2.0" upper="2.0" effort="100" velocity="1.0"/>
+  </joint>
+  <!-- Base Y → Base Link (prismatic joint for z-axis motion) -->
+  <joint name="joint_base_y_to_base_z" type="prismatic">
+        <origin xyz="0 0 0" rpy="0 0 0"/>
+        <parent link="base_link_y_frame"/>
         <child link="base_link"/>
-    </joint>
+        <axis xyz="0 0 1"/>
+        <limit lower="0.0" upper="2.0" effort="100" velocity="1.0"/>
+  </joint>
   <!-- Base → Wrist -->
   <joint name="joint_base_to_wrist" type="fixed">
     <parent link="base_link"/>
     <child  link="wrist_link"/>
-    <origin xyz="${base_length} 0 ${base_depth/2}" rpy="0 0 0"/>
+    <origin xyz="${base_length/2} 0 0" rpy="0 0 0"/>
   </joint>
   <!-- Wrist → Palm -->

Commit message: Searching for the sensor problem. Still no publishing in dedicated topic

File: ros2_ws/src/prosthesis_description/model/gazebo.xacro (robot description, xacro)
@@ -1,5 +1,5 @@
 <?xml version="1.0"?>
-<robot xmlns:xacro="http://www.ros.org/wiki/xacro">
-<!-- File containing all additional descriptions necessary for Gazebo simulation-->
+<robot name="prosthesis" xmlns:xacro="http://www.ros.org/wiki/xacro">
+  <!-- File containing all additional descriptions necessary for Gazebo simulation-->
   <!-- ===== GAZEBO TAGS ROS2 CONTROL PLUGIN ===== -->
   <!-- Needed additional link properties to simulate robot in accurate physics environment-->
@@ -10,7 +10,26 @@
     <plugin filename="gz_ros2_control-system" name="gz_ros2_control::GazeboSimROS2ControlPlugin">
       <parameters>$(find prosthesis_description)/config/prosthesis_controllers.yaml</parameters>
-      <controller_manager_prefix_node_name>controller_manager</controller_manager_prefix_node_name>
+      <!--<controller_manager_prefix_node_name>controller_manager</controller_manager_prefix_node_name>-->
     </plugin>
   </gazebo>
+  <gazebo>
+      <plugin
+          filename="gz-sim-joint-state-publisher-system"
+          name="gz::sim::systems::JointStatePublisher">
+          <topic>joint_states</topic>
+          <joint_name>joint_wrist_to_palm</joint_name>
+          <joint_name>joint_index_mcp</joint_name>
+          <joint_name>joint_index_pip</joint_name>
+          <joint_name>joint_middle_mcp</joint_name>
+          <joint_name>joint_middle_pip</joint_name>
+          <joint_name>joint_ring_mcp</joint_name>
+          <joint_name>joint_ring_pip</joint_name>
+          <joint_name>joint_little_mcp</joint_name>
+          <joint_name>joint_little_pip</joint_name>
+          <joint_name>joint_thumb_cmc</joint_name>
+          <joint_name>joint_thumb_mcp</joint_name>
+          <joint_name>joint_thumb_pip</joint_name>
+      </plugin>
+    </gazebo>
   <!-- Base and palm Gazebo tags -->
   <gazebo reference="base_link">
@@ -154,8 +173,8 @@
     <sensor name="index_fsr" type="contact">
       <always_on>true</always_on>
-      <update_rate>1000</update_rate>
-      <plugin filename="gz-sim-contact-system" name="gz::sim::systems::Contact" />
-      <contact>
-        <collision>collision</collision>
+      <update_rate>100</update_rate>
+      <contact>
+        <collision>collision_index_middle_fsr</collision>
+        <topic>/index_fsr</topic>
       </contact>
     </sensor>
@@ -164,7 +183,8 @@
       <sensor name="middle_fsr" type="contact">
       <always_on>true</always_on>
-      <update_rate>1000</update_rate>
-      <contact>
-        <collision>collision</collision>
+      <update_rate>100</update_rate>
+      <contact>
+        <collision>collision_middle_middle</collision>
+        <topic>/middle_fsr</topic>
       </contact>
     </sensor>
@@ -173,7 +193,8 @@
     <sensor name="ring_fsr" type="contact">
       <always_on>true</always_on>
-      <update_rate>1000</update_rate>
-      <contact>
-        <collision>collision</collision>
+      <update_rate>100</update_rate>
+      <contact>
+        <collision>collision_ring_middle</collision>
+        <topic>/ring_fsr</topic>
       </contact>
     </sensor>
@@ -182,7 +203,8 @@
     <sensor name="little_fsr" type="contact">
       <always_on>true</always_on>
-      <update_rate>1000</update_rate>
-      <contact>
-        <collision>collision</collision>
+      <update_rate>100</update_rate>
+      <contact>
+        <collision>collision_little_middle</collision>
+        <topic>/little_fsr</topic>
       </contact>
     </sensor>
@@ -191,99 +213,46 @@
     <sensor name="thumb_fsr" type="contact">
       <always_on>true</always_on>
-      <update_rate>1000</update_rate>
-      <contact>
-        <collision>collision</collision>
-      </contact>
-    </sensor>
-  </gazebo>
-  <!-- ===== ROS2 CONTROL INTERFACE ===== -->
-  <!-- Tells control_manager what hardware plugin to instanciate,
-   which joint exists and which interface each joint exposes -->
-  <ros2_control name="GazeboSimROS2ControlPlugin" type="system">
-    <hardware>
-      <plugin>gz_ros2_control/GazeboSimSystem</plugin>
-    </hardware>
-    <!-- Base Movement Joints (X, Y, Z) -->
-    <joint name="joint_world_to_base_x">
-      <command_interface name="position"/>
-      <state_interface name="position"/>
-      <state_interface name="velocity"/>
-    </joint>
-    <joint name="joint_base_x_to_base_y">
-      <command_interface name="position"/>
-      <state_interface name="position"/>
-      <state_interface name="velocity"/>
-    </joint>
-    <joint name="joint_base_y_to_base_z">
-      <command_interface name="position"/>
-      <state_interface name="position"/>
-      <state_interface name="velocity"/>
-    </joint>
-    <!-- Wrist Joint -->
-    <joint name="joint_wrist_to_palm">
-      <command_interface name="position"/> <!-- command controller will send for position control -->
-      <state_interface name="position"/> <!-- state controller can read -->
-      <state_interface name="velocity"/>
-    </joint>
-    <!-- Index Finger Joints -->
-    <joint name="joint_index_mcp">
-      <command_interface name="position"/>
-      <state_interface name="position"/>
-      <state_interface name="velocity"/>
-    </joint>
-    <joint name="joint_index_pip">
-      <command_interface name="position"/>
-      <state_interface name="position"/>
-      <state_interface name="velocity"/>
-    </joint>
-    <!-- Middle Finger Joints -->
-    <joint name="joint_middle_mcp">
-      <command_interface name="position"/>
-      <state_interface name="position"/>
-      <state_interface name="velocity"/>
-    </joint>
-    <joint name="joint_middle_pip">
-      <command_interface name="position"/>
-      <state_interface name="position"/>
-      <state_interface name="velocity"/>
-    </joint>
-    <!-- Ring Finger Joints -->
-    <joint name="joint_ring_mcp">
-      <command_interface name="position"/>
-      <state_interface name="position"/>
-      <state_interface name="velocity"/>
-    </joint>
-    <joint name="joint_ring_pip">
-      <command_interface name="position"/>
-      <state_interface name="position"/>
-      <state_interface name="velocity"/>
-    </joint>
-    <!-- Little Finger Joints -->
-    <joint name="joint_little_mcp">
-      <command_interface name="position"/>
-      <state_interface name="position"/>
-      <state_interface name="velocity"/>
-    </joint>
-    <joint name="joint_little_pip">
-      <command_interface name="position"/>
-      <state_interface name="position"/>
-      <state_interface name="velocity"/>
-    </joint>
-    <!-- Thumb Joints -->
-    <joint name="joint_thumb_cmc">
-      <command_interface name="position"/>
-      <state_interface name="position"/>
-      <state_interface name="velocity"/>
-    </joint>
-    <joint name="joint_thumb_mcp">
-      <command_interface name="position"/>
-      <state_interface name="position"/>
-      <state_interface name="velocity"/>
-    </joint>
-    <joint name="joint_thumb_ip">
-      <command_interface name="position"/>
-      <state_interface name="position"/>
-      <state_interface name="velocity"/>
-    </joint>
-  </ros2_control>
+      <update_rate>100</update_rate>
+      <contact>
+        <collision>collision_thumb_distal</collision>
+        <topic>/thumb_fsr</topic>
+      </contact>
+    </sensor>
+  </gazebo>
+  <!-- Force-torque sensor -->
+  <gazebo reference="joint_index_mcp">
+    <sensor name="index_ft" type="force_torque">
+      <always_on>true</always_on>
+      <update_rate>100</update_rate>
+      <pose>0 0 0 0 0 0</pose>
+    </sensor>
+  </gazebo>
+  <gazebo reference="joint_middle_mcp">
+    <sensor name="middle_ft" type="force_torque">
+      <always_on>true</always_on>
+      <update_rate>100</update_rate>
+      <pose>0 0 0 0 0 0</pose>
+    </sensor>
+  </gazebo>
+  <gazebo reference="joint_ring_mcp">
+    <sensor name="ring_ft" type="force_torque">
+      <always_on>true</always_on>
+      <update_rate>100</update_rate>
+      <pose>0 0 0 0 0 0</pose>
+    </sensor>
+  </gazebo>
+  <gazebo reference="joint_little_mcp">
+    <sensor name="little_ft" type="force_torque">
+      <always_on>true</always_on>
+      <update_rate>100</update_rate>
+      <pose>0 0 0 0 0 0</pose>
+    </sensor>
+  </gazebo>
+  <gazebo reference="joint_thumb_cmc">
+    <sensor name="thumb_ft" type="force_torque">
+      <always_on>true</always_on>
+      <update_rate>100</update_rate>
+      <pose>0 0 0 0 0 0</pose>
+    </sensor>
+  </gazebo>
 </robot>

File: ros2_ws/src/prosthesis_description/model/parameters.xacro (robot description, xacro)
@@ -1,5 +1,5 @@
 <?xml version="1.0"?>
-<robot xmlns:xacro="http://www.ros.org/wiki/xacro" >
-<!-- File containing all useful values for the robot description -->
+<robot name="prosthesis" xmlns:xacro="http://www.ros.org/wiki/xacro">
+    <!-- File containing all useful values for the robot description -->
     <!-- ==== PROSTHESIS VALUES ==== -->
     <!-- Dimensions for each link -->
