Commit message: Working FSR sensors !!!!!!!!!!!!!!

File: ros2_ws/src/prosthesis_description/model/gazebo.xacro (robot description, xacro)
@@ -175,5 +175,5 @@
       <update_rate>100</update_rate>
       <contact>
-        <collision>collision_index_middle_fsr</collision>
+        <collision>index_middle_fsr_link_collision</collision>
         <topic>/index_fsr</topic>
       </contact>
@@ -185,5 +185,5 @@
       <update_rate>100</update_rate>
       <contact>
-        <collision>collision_middle_middle</collision>
+        <collision>middle_middle_link_collision</collision>
         <topic>/middle_fsr</topic>
       </contact>
@@ -195,5 +195,5 @@
       <update_rate>100</update_rate>
       <contact>
-        <collision>collision_ring_middle</collision>
+        <collision>ring_middle_link_collision</collision>
         <topic>/ring_fsr</topic>
       </contact>
@@ -205,5 +205,5 @@
       <update_rate>100</update_rate>
       <contact>
-        <collision>collision_little_middle</collision>
+        <collision>little_middle_link_collision</collision>
         <topic>/little_fsr</topic>
       </contact>
@@ -215,5 +215,5 @@
       <update_rate>100</update_rate>
       <contact>
-        <collision>collision_thumb_distal</collision>
+        <collision>thumb_distal_link_collision</collision>
         <topic>/thumb_fsr</topic>
       </contact>

File: ros2_ws/src/prosthesis_description/model/prosthesis.urdf.xacro (robot description, xacro)
@@ -67,5 +67,5 @@
           <geometry><box size="${index_proximal_length} ${index_proximal_width} ${index_proximal_depth}"/></geometry>
       </visual>
-      <collision name="collision_index_proximal">
+      <collision>
           <origin xyz="${index_proximal_length/2} 0 0" rpy="0 0 0"/>
           <geometry><box size="${index_proximal_length} ${index_proximal_width} ${index_proximal_depth}"/></geometry>
@@ -80,5 +80,5 @@
           <geometry><box size="${index_middle_length} ${index_middle_width} ${index_middle_depth}"/></geometry>
       </visual>
-      <collision name="collision_index_middle">
+      <collision>
           <origin xyz="${index_middle_length/2} 0 0" rpy="0 0 0"/>
           <geometry><box size="${index_middle_length} ${index_middle_width} ${index_middle_depth}"/></geometry>
@@ -93,5 +93,5 @@
           <geometry><sphere radius="0.005"/></geometry>
       </visual>
-      <collision name="collision_index_middle_fsr">
+      <collision>
           <origin xyz="${index_middle_length/2} 0 0" rpy="0 0 0"/>
           <geometry><sphere radius="0.005"/></geometry>
@@ -123,5 +123,5 @@
           <geometry><box size="${middle_middle_length} ${middle_middle_width} ${middle_middle_depth}"/></geometry>
       </visual>
-      <collision name="collision_middle_middle">
+      <collision>
           <origin xyz="${middle_middle_length/2} 0 0" rpy="0 0 0"/>
           <geometry><box size="${middle_middle_length} ${middle_middle_width} ${middle_middle_depth}"/></geometry>
@@ -137,5 +137,5 @@
           <geometry><box size="${ring_proximal_length} ${ring_proximal_width} ${ring_proximal_depth}"/></geometry>
       </visual>
-      <collision name="collision_ring_proximal">
+      <collision>
           <origin xyz="${ring_proximal_length/2} 0 0" rpy="0 0 0"/>
           <geometry><box size="${ring_proximal_length} ${ring_proximal_width} ${ring_proximal_depth}"/></geometry>
@@ -150,5 +150,5 @@
           <geometry><box size="${ring_middle_length} ${ring_middle_width} ${ring_middle_depth}"/></geometry>
       </visual>
-      <collision name="collision_ring_middle">
+      <collision>
           <origin xyz="${ring_middle_length/2} 0 0" rpy="0 0 0"/>
           <geometry><box size="${ring_middle_length} ${ring_middle_width} ${ring_middle_depth}"/></geometry>
@@ -164,5 +164,5 @@
           <geometry><box size="${little_proximal_length} ${little_proximal_width} ${little_proximal_depth}"/></geometry>
       </visual>
-      <collision name="collision_little_proximal">
+      <collision>
           <origin xyz="${little_proximal_length/2} 0 0" rpy="0 0 0"/>
           <geometry><box size="${little_proximal_length} ${little_proximal_width} ${little_proximal_depth}"/></geometry>
@@ -177,5 +177,5 @@
           <geometry><box size="${little_middle_length} ${little_middle_width} ${little_middle_depth}"/></geometry>
       </visual>
-      <collision name="collision_little_middle">
+      <collision>
           <origin xyz="${little_middle_length/2} 0 0" rpy="0 0 0"/>
           <geometry><box size="${little_middle_length} ${little_middle_width} ${little_middle_depth}"/></geometry>
@@ -191,5 +191,5 @@
           <geometry><box size="${thumb_metacarpal_length} ${thumb_metacarpal_width} ${thumb_metacarpal_depth}"/></geometry>
       </visual>
-      <collision name="collision_thumb_metacarpal">
+      <collision>
           <origin xyz="${thumb_metacarpal_length/2} 0 0" rpy="0 0 0"/>
           <geometry><box size="${thumb_metacarpal_length} ${thumb_metacarpal_width} ${thumb_metacarpal_depth}"/></geometry>
@@ -204,5 +204,5 @@
           <geometry><box size="${thumb_proximal_length} ${thumb_proximal_width} ${thumb_proximal_depth}"/></geometry>
       </visual>
-      <collision name="collision_thumb_proximal">
+      <collision>
           <origin xyz="${thumb_proximal_length/2} 0 0" rpy="0 0 0"/>
           <geometry><box size="${thumb_proximal_length} ${thumb_proximal_width} ${thumb_proximal_depth}"/></geometry>
@@ -217,5 +217,5 @@
           <geometry><box size="${thumb_distal_length} ${thumb_distal_width} ${thumb_distal_depth}"/></geometry>
       </visual>
-      <collision name="collision_thumb_distal">
+      <collision>
           <origin xyz="${thumb_distal_length/2} 0 0" rpy="0 0 0"/>
           <geometry><box size="${thumb_distal_length} ${thumb_distal_width} ${thumb_distal_depth}"/></geometry>

Commit message: Started mesh integration and implementing finger dynamism

File: ros2_ws/src/prosthesis_description/model/gazebo.xacro (robot description, xacro)
@@ -19,6 +19,8 @@
           <topic>joint_states</topic>
           <joint_name>joint_wrist_to_palm</joint_name>
-          <joint_name>joint_index_mcp</joint_name>
-          <joint_name>joint_index_pip</joint_name>
+          <joint_name>joint_index_1</joint_name>
+          <joint_name>joint_index_2</joint_name>
+          <joint_name>joint_index_3</joint_name>
+          <joint_name>joint_index_4</joint_name>
           <joint_name>joint_middle_mcp</joint_name>
           <joint_name>joint_middle_pip</joint_name>
@@ -59,15 +61,33 @@
   </gazebo>
   <!-- Index finger Gazebo tags -->
-  <gazebo reference="index_proximal_link">
-    <material>Gazebo/SkyBlue</material>
-    <mu1>${palm_fingers_friction}</mu1>
-    <mu2>${palm_fingers_friction}</mu2>
-    <kp>${rigid_stiffness_default}</kp>
-    <kd>${damping_default}</kd>
-    <minDepth>${min_depth_default}</minDepth>
-    <maxVel>${max_velocity_default}</maxVel>
-  </gazebo>
-  <gazebo reference="index_middle_link">
-    <material>Gazebo/Blue</material>
+  <gazebo reference="link_index_1">
+    <material>Gazebo/Blue</material>
+    <mu1>${palm_fingers_friction}</mu1>
+    <mu2>${palm_fingers_friction}</mu2>
+    <kp>${rigid_stiffness_default}</kp>
+    <kd>${damping_default}</kd>
+    <minDepth>${min_depth_default}</minDepth>
+    <maxVel>${max_velocity_default}</maxVel>
+  </gazebo>
+  <gazebo reference="link_index_2">
+    <material>Gazebo/Red</material>
+    <mu1>${palm_fingers_friction}</mu1>
+    <mu2>${palm_fingers_friction}</mu2>
+    <kp>${rigid_stiffness_default}</kp>
+    <kd>${damping_default}</kd>
+    <minDepth>${min_depth_default}</minDepth>
+    <maxVel>${max_velocity_default}</maxVel>
+  </gazebo>
+  <gazebo reference="link_index_3">
+    <material>Gazebo/Blue</material>
+    <mu1>${palm_fingers_friction}</mu1>
+    <mu2>${palm_fingers_friction}</mu2>
+    <kp>${rigid_stiffness_default}</kp>
+    <kd>${damping_default}</kd>
+    <minDepth>${min_depth_default}</minDepth>
+    <maxVel>${max_velocity_default}</maxVel>
+  </gazebo>
+  <gazebo reference="link_index_4">
+    <material>Gazebo/Red</material>
     <mu1>${palm_fingers_friction}</mu1>
     <mu2>${palm_fingers_friction}</mu2>
@@ -221,5 +241,5 @@
   </gazebo>
   <!-- Force-torque sensor -->
-  <gazebo reference="joint_index_mcp">
+  <gazebo reference="joint_index_1">
     <sensor name="prosthesis/sensor/index_ft" type="force_torque">
       <always_on>true</always_on>

File: ros2_ws/src/prosthesis_description/model/prosthesis.urdf.xacro (robot description, xacro)
@@ -23,7 +23,5 @@
       <visual>
           <origin xyz="0 0 0" rpy="0 0 0"/>
-          <geometry>
-            <mesh filename="$(find prosthesis_description)/meshes/PhalangeConstructrion_Base.stl" />
-          </geometry>
+          <geometry><box size="${base_length} ${base_width} ${base_depth}"/></geometry>
       </visual>
       <collision>
@@ -64,12 +62,14 @@
     <!-- ===== FINGER & THUMB LINKS (all boxes 0.02 x 0.05 x 0.02) ===== -->
     <!-- Index -->
-    <link name="index_proximal_link">
-      <visual>
-          <origin xyz="${index_proximal_length/2} 0 0" rpy="0 0 0"/>
-          <geometry><box size="${index_proximal_length} ${index_proximal_width} ${index_proximal_depth}"/></geometry>
-      </visual>
-      <collision>
-          <origin xyz="${index_proximal_length/2} 0 0" rpy="0 0 0"/>
-          <geometry><box size="${index_proximal_length} ${index_proximal_width} ${index_proximal_depth}"/></geometry>
+    <link name="link_index_1">
+      <visual>
+          <origin xyz="0 0 0" rpy="0 0 0"/>
+          <geometry><mesh filename="$(find prosthesis_description)/meshes/PhalangeConstruction_Part_3.stl"/></geometry>
+      </visual>
+      <collision>
+          <origin xyz="0 0 0" rpy="0 0 0"/>
+          <geometry><mesh filename="$(find prosthesis_description)/meshes/PhalangeConstruction_Part_3.stl"/></geometry>
+          <!--<origin xyz="${index_proximal_length/2} 0 0" rpy="0 0 0"/>
+          <geometry><box size="${index_proximal_length} ${index_proximal_width} ${index_proximal_depth}"/></geometry>-->
       </collision>
       <xacro:inertial_box mass="0.01" x="${index_proximal_length}" y="${index_proximal_width}" z="${index_proximal_depth}">
@@ -77,12 +77,42 @@
       </xacro:inertial_box>
     </link>
-    <link name="index_middle_link">
-      <visual>
+    <link name="link_index_2">
+      <visual>
+          <!--<origin xyz="0 0 0" rpy="0 0 0"/>
+          <geometry><mesh filename="$(find prosthesis_description)/meshes/PhalangeConstruction_Part_4.stl"/></geometry>-->
+          <origin xyz="${index_middle_length/2} 0 0" rpy="0 0 0"/>
+          <geometry><box size="${index_middle_length/4} ${index_middle_width} ${index_middle_depth}"/></geometry>
+      </visual>
+      <collision>
+          <!--<origin xyz="0 0 0" rpy="0 0 0"/>
+          <geometry><mesh filename="$(find prosthesis_description)/meshes/PhalangeConstruction_Part_4.stl"/></geometry>-->
           <origin xyz="${index_middle_length/2} 0 0" rpy="0 0 0"/>
           <geometry><box size="${index_middle_length} ${index_middle_width} ${index_middle_depth}"/></geometry>
-      </visual>
-      <collision>
-          <origin xyz="${index_middle_length/2} 0 0" rpy="0 0 0"/>
-          <geometry><box size="${index_middle_length} ${index_middle_width} ${index_middle_depth}"/></geometry>
+      </collision>
+      <xacro:inertial_box mass="0.02" x="${index_middle_length}" y="${index_middle_width}" z="${index_middle_depth}">
+          <origin xyz="${index_middle_length/2} 0 0" rpy="0 0 0"/>
+      </xacro:inertial_box>
+    </link>
+    <link name="link_index_3">
+      <visual>
+          <origin xyz="0 0 0" rpy="0 0 0"/>
+          <geometry><mesh filename="$(find prosthesis_description)/meshes/PhalangeConstruction_Part_5.stl"/></geometry>
+      </visual>
+      <collision>
+          <origin xyz="0 0 0" rpy="0 0 0"/>
+          <geometry><mesh filename="$(find prosthesis_description)/meshes/PhalangeConstruction_Part_5.stl"/></geometry>
+      </collision>
+      <xacro:inertial_box mass="0.02" x="${index_middle_length}" y="${index_middle_width}" z="${index_middle_depth}">
+          <origin xyz="${index_middle_length/2} 0 0" rpy="0 0 0"/>
+      </xacro:inertial_box>
+    </link>
+    <link name="link_index_4">
+      <visual>
+          <origin xyz="0 0 0" rpy="-1.57 0 0"/>
+          <geometry><mesh filename="$(find prosthesis_description)/meshes/PhalangeConstruction_Part_6.stl"/></geometry>
+      </visual>
+      <collision>
+          <origin xyz="0 0 0" rpy="-1.57 0 0"/>
+          <geometry><mesh filename="$(find prosthesis_description)/meshes/PhalangeConstruction_Part_6.stl"/></geometry>
       </collision>
       <xacro:inertial_box mass="0.02" x="${index_middle_length}" y="${index_middle_width}" z="${index_middle_depth}">
@@ -268,16 +298,26 @@
     </joint>
     <!-- Index -->
-    <joint name="joint_index_mcp" type="revolute">
-      <parent link="palm_link"/><child link="index_proximal_link"/>
+    <joint name="joint_index_1" type="revolute">
+      <parent link="palm_link"/><child link="link_index_1"/>
       <origin xyz="${mcp_x} ${index_mcp_y} 0.0" rpy="0 0 0"/><axis xyz="0 1 0"/>
       <limit lower="0.0" upper="1.57" effort="3" velocity="5"/>
     </joint>
-    <joint name="joint_index_pip" type="revolute">
-      <parent link="index_proximal_link"/><child link="index_middle_link"/>
+    <joint name="joint_index_2" type="revolute">
+      <parent link="link_index_1"/><child link="link_index_2"/>
       <origin xyz="${index_proximal_length} 0 0" rpy="0 0 0"/><axis xyz="0 1 0"/>
       <limit lower="0.0" upper="1.57" effort="2" velocity="5"/>
     </joint>
+    <joint name="joint_index_3" type="revolute">
+      <parent link="link_index_2"/><child link="link_index_3"/>
+      <origin xyz="${index_proximal_length} 0 0" rpy="0 0 0"/><axis xyz="0 1 0"/>
+      <limit lower="0.0" upper="1.57" effort="2" velocity="5"/>
+    </joint>
+    <joint name="joint_index_4" type="revolute">
+      <parent link="link_index_3"/><child link="link_index_4"/>
+      <origin xyz="${index_proximal_length} 0 0" rpy="0 0 0"/><axis xyz="0 1 0"/>
+      <limit lower="0.0" upper="1.57" effort="2" velocity="5"/>
+    </joint>
     <joint name="joint_index_fsr" type="fixed">
-      <parent link="index_middle_link"/><child link="index_middle_fsr_link"/>
+      <parent link="link_index_4"/><child link="index_middle_fsr_link"/>
       <origin xyz="${index_middle_length/2} 0 0" rpy="0 0 0"/>
     </joint>
@@ -365,11 +405,23 @@
     </joint>
     <!-- Index Finger Joints -->
-    <joint name="joint_index_mcp">
-      <command_interface name="position"/>
-      <state_interface name="position"/>
-      <state_interface name="velocity"/>
-      <state_interface name="effort"/>
-    </joint>
-    <joint name="joint_index_pip">
+    <joint name="joint_index_1">
+      <command_interface name="position"/>
+      <state_interface name="position"/>
+      <state_interface name="velocity"/>
+      <state_interface name="effort"/>
+    </joint>
+    <joint name="joint_index_2">
+      <command_interface name="position"/>
+      <state_interface name="position"/>
+      <state_interface name="velocity"/>
+      <state_interface name="effort"/>
+    </joint>
+    <joint name="joint_index_3">
+      <command_interface name="position"/>
+      <state_interface name="position"/>
+      <state_interface name="velocity"/>
+      <state_interface name="effort"/>
+    </joint>
+      <joint name="joint_index_4">
       <command_interface name="position"/>
       <state_interface name="position"/>
