Commit message: Added meshes to fingers (still need to be adjusted) Also trajectory_goals for keyboard control need to be adjusted (too big mouvements, not easily controllable)

File: ros2_ws/src/prosthesis_description/model/gazebo.xacro (robot description, xacro)
@@ -23,13 +23,19 @@
           <joint_name>joint_index_3</joint_name>
           <joint_name>joint_index_4</joint_name>
-          <joint_name>joint_middle_mcp</joint_name>
-          <joint_name>joint_middle_pip</joint_name>
-          <joint_name>joint_ring_mcp</joint_name>
-          <joint_name>joint_ring_pip</joint_name>
-          <joint_name>joint_little_mcp</joint_name>
-          <joint_name>joint_little_pip</joint_name>
-          <joint_name>joint_thumb_cmc</joint_name>
-          <joint_name>joint_thumb_mcp</joint_name>
-          <joint_name>joint_thumb_pip</joint_name>
+          <joint_name>joint_middle_1</joint_name>
+          <joint_name>joint_middle_2</joint_name>
+          <joint_name>joint_middle_3</joint_name>
+          <joint_name>joint_middle_4</joint_name>
+          <joint_name>joint_ring_1</joint_name>
+          <joint_name>joint_ring_2</joint_name>
+          <joint_name>joint_ring_3</joint_name>
+          <joint_name>joint_ring_4</joint_name>
+          <joint_name>joint_little_1</joint_name>
+          <joint_name>joint_little_2</joint_name>
+          <joint_name>joint_little_3</joint_name>
+          <joint_name>joint_little_4</joint_name>
+          <joint_name>joint_thumb_1</joint_name>
+          <joint_name>joint_thumb_2</joint_name>
+          <joint_name>joint_thumb_3</joint_name>
       </plugin>
     </gazebo>
@@ -98,15 +104,33 @@
   </gazebo>
   <!-- Middle finger Gazebo tags -->
-  <gazebo reference="middle_proximal_link">
-    <material>Gazebo/SkyBlue</material>
-    <mu1>${palm_fingers_friction}</mu1>
-    <mu2>${palm_fingers_friction}</mu2>
-    <kp>${rigid_stiffness_default}</kp>
-    <kd>${damping_default}</kd>
-    <minDepth>${min_depth_default}</minDepth>
-    <maxVel>${max_velocity_default}</maxVel>
-  </gazebo>
-  <gazebo reference="middle_middle_link">
-    <material>Gazebo/Blue</material>
+  <gazebo reference="link_middle_1">
+    <material>Gazebo/Blue</material>
+    <mu1>${palm_fingers_friction}</mu1>
+    <mu2>${palm_fingers_friction}</mu2>
+    <kp>${rigid_stiffness_default}</kp>
+    <kd>${damping_default}</kd>
+    <minDepth>${min_depth_default}</minDepth>
+    <maxVel>${max_velocity_default}</maxVel>
+  </gazebo>
+  <gazebo reference="link_middle_2">
+    <material>Gazebo/Red</material>
+    <mu1>${palm_fingers_friction}</mu1>
+    <mu2>${palm_fingers_friction}</mu2>
+    <kp>${rigid_stiffness_default}</kp>
+    <kd>${damping_default}</kd>
+    <minDepth>${min_depth_default}</minDepth>
+    <maxVel>${max_velocity_default}</maxVel>
+  </gazebo>
+  <gazebo reference="link_middle_3">
+    <material>Gazebo/Blue</material>
+    <mu1>${palm_fingers_friction}</mu1>
+    <mu2>${palm_fingers_friction}</mu2>
+    <kp>${rigid_stiffness_default}</kp>
+    <kd>${damping_default}</kd>
+    <minDepth>${min_depth_default}</minDepth>
+    <maxVel>${max_velocity_default}</maxVel>
+  </gazebo>
+  <gazebo reference="link_middle_4">
+    <material>Gazebo/Red</material>
     <mu1>${palm_fingers_friction}</mu1>
     <mu2>${palm_fingers_friction}</mu2>
@@ -117,15 +141,33 @@
   </gazebo>
   <!-- Ring finger Gazebo tags -->
-  <gazebo reference="ring_proximal_link">
-    <material>Gazebo/SkyBlue</material>
-    <mu1>${palm_fingers_friction}</mu1>
-    <mu2>${palm_fingers_friction}</mu2>
-    <kp>${rigid_stiffness_default}</kp>
-    <kd>${damping_default}</kd>
-    <minDepth>${min_depth_default}</minDepth>
-    <maxVel>${max_velocity_default}</maxVel>
-  </gazebo>
-  <gazebo reference="ring_middle_link">
-    <material>Gazebo/Blue</material>
+  <gazebo reference="link_ring_1">
+    <material>Gazebo/Blue</material>
+    <mu1>${palm_fingers_friction}</mu1>
+    <mu2>${palm_fingers_friction}</mu2>
+    <kp>${rigid_stiffness_default}</kp>
+    <kd>${damping_default}</kd>
+    <minDepth>${min_depth_default}</minDepth>
+    <maxVel>${max_velocity_default}</maxVel>
+  </gazebo>
+  <gazebo reference="link_ring_2">
+    <material>Gazebo/Red</material>
+    <mu1>${palm_fingers_friction}</mu1>
+    <mu2>${palm_fingers_friction}</mu2>
+    <kp>${rigid_stiffness_default}</kp>
+    <kd>${damping_default}</kd>
+    <minDepth>${min_depth_default}</minDepth>
+    <maxVel>${max_velocity_default}</maxVel>
+  </gazebo>
+  <gazebo reference="link_ring_3">
+    <material>Gazebo/Blue</material>
+    <mu1>${palm_fingers_friction}</mu1>
+    <mu2>${palm_fingers_friction}</mu2>
+    <kp>${rigid_stiffness_default}</kp>
+    <kd>${damping_default}</kd>
+    <minDepth>${min_depth_default}</minDepth>
+    <maxVel>${max_velocity_default}</maxVel>
+  </gazebo>
+  <gazebo reference="link_ring_4">
+    <material>Gazebo/Red</material>
     <mu1>${palm_fingers_friction}</mu1>
     <mu2>${palm_fingers_friction}</mu2>
@@ -136,15 +178,33 @@
   </gazebo>
   <!-- Little finger Gazebo tags -->
-  <gazebo reference="little_proximal_link">
-    <material>Gazebo/SkyBlue</material>
-    <mu1>${palm_fingers_friction}</mu1>
-    <mu2>${palm_fingers_friction}</mu2>
-    <kp>${rigid_stiffness_default}</kp>
-    <kd>${damping_default}</kd>
-    <minDepth>${min_depth_default}</minDepth>
-    <maxVel>${max_velocity_default}</maxVel>
-  </gazebo>
-  <gazebo reference="little_middle_link">
-    <material>Gazebo/Blue</material>
+  <gazebo reference="link_little_1">
+    <material>Gazebo/Blue</material>
+    <mu1>${palm_fingers_friction}</mu1>
+    <mu2>${palm_fingers_friction}</mu2>
+    <kp>${rigid_stiffness_default}</kp>
+    <kd>${damping_default}</kd>
+    <minDepth>${min_depth_default}</minDepth>
+    <maxVel>${max_velocity_default}</maxVel>
+  </gazebo>
+  <gazebo reference="link_little_2">
+    <material>Gazebo/Red</material>
+    <mu1>${palm_fingers_friction}</mu1>
+    <mu2>${palm_fingers_friction}</mu2>
+    <kp>${rigid_stiffness_default}</kp>
+    <kd>${damping_default}</kd>
+    <minDepth>${min_depth_default}</minDepth>
+    <maxVel>${max_velocity_default}</maxVel>
+  </gazebo>
+  <gazebo reference="link_little_3">
+    <material>Gazebo/Blue</material>
+    <mu1>${palm_fingers_friction}</mu1>
+    <mu2>${palm_fingers_friction}</mu2>
+    <kp>${rigid_stiffness_default}</kp>
+    <kd>${damping_default}</kd>
+    <minDepth>${min_depth_default}</minDepth>
+    <maxVel>${max_velocity_default}</maxVel>
+  </gazebo>
+  <gazebo reference="link_little_4">
+    <material>Gazebo/Red</material>
     <mu1>${palm_fingers_friction}</mu1>
     <mu2>${palm_fingers_friction}</mu2>
@@ -155,24 +215,24 @@
   </gazebo>
   <!-- Thumb Gazebo tags -->
-  <gazebo reference="thumb_metacarpal_link">
-    <material>Gazebo/Green</material>
-    <mu1>${palm_fingers_friction}</mu1>
-    <mu2>${palm_fingers_friction}</mu2>
-    <kp>${rigid_stiffness_default}</kp>
-    <kd>${damping_default}</kd>
-    <minDepth>${min_depth_default}</minDepth>
-    <maxVel>${max_velocity_default}</maxVel>
-  </gazebo>
-  <gazebo reference="thumb_proximal_link">
-    <material>Gazebo/Green</material>
-    <mu1>${palm_fingers_friction}</mu1>
-    <mu2>${palm_fingers_friction}</mu2>
-    <kp>${rigid_stiffness_default}</kp>
-    <kd>${damping_default}</kd>
-    <minDepth>${min_depth_default}</minDepth>
-    <maxVel>${max_velocity_default}</maxVel>
-  </gazebo>
-  <gazebo reference="thumb_distal_link">
-    <material>Gazebo/Green</material>
+  <gazebo reference="link_thumb_1">
+    <material>Gazebo/Blue</material>
+    <mu1>${palm_fingers_friction}</mu1>
+    <mu2>${palm_fingers_friction}</mu2>
+    <kp>${rigid_stiffness_default}</kp>
+    <kd>${damping_default}</kd>
+    <minDepth>${min_depth_default}</minDepth>
+    <maxVel>${max_velocity_default}</maxVel>
+  </gazebo>
+  <gazebo reference="link_thumb_2">
+    <material>Gazebo/Red</material>
+    <mu1>${palm_fingers_friction}</mu1>
+    <mu2>${palm_fingers_friction}</mu2>
+    <kp>${rigid_stiffness_default}</kp>
+    <kd>${damping_default}</kd>
+    <minDepth>${min_depth_default}</minDepth>
+    <maxVel>${max_velocity_default}</maxVel>
+  </gazebo>
+  <gazebo reference="link_thumb_3">
+    <material>Gazebo/Blue</material>
     <mu1>${palm_fingers_friction}</mu1>
     <mu2>${palm_fingers_friction}</mu2>
@@ -200,40 +260,40 @@
     </sensor>
   </gazebo>
-  <gazebo reference="middle_middle_link">
+  <gazebo reference="link_middle_4">
       <sensor name="middle_fsr" type="contact">
       <always_on>true</always_on>
       <update_rate>100</update_rate>
       <contact>
-        <collision>middle_middle_link_collision</collision>
+        <collision>link_middle_4_collision</collision>
         <topic>prosthesis/sensor/middle_fsr</topic>
       </contact>
     </sensor>
   </gazebo>
-  <gazebo reference="ring_middle_link">
+  <gazebo reference="link_ring_4">
     <sensor name="ring_fsr" type="contact">
       <always_on>true</always_on>
       <update_rate>100</update_rate>
       <contact>
-        <collision>ring_middle_link_collision</collision>
+        <collision>link_ring_4_collision</collision>
         <topic>prosthesis/sensor/ring_fsr</topic>
       </contact>
     </sensor>
   </gazebo>
-  <gazebo reference="little_middle_link">
+  <gazebo reference="link_little_4">
     <sensor name="little_fsr" type="contact">
       <always_on>true</always_on>
       <update_rate>100</update_rate>
       <contact>
-        <collision>little_middle_link_collision</collision>
+        <collision>link_little_4_collision</collision>
         <topic>prosthesis/sensor/little_fsr</topic>
       </contact>
     </sensor>
   </gazebo>
-  <gazebo reference="thumb_distal_link">
+  <gazebo reference="link_thumb_3">
     <sensor name="thumb_fsr" type="contact">
       <always_on>true</always_on>
       <update_rate>100</update_rate>
       <contact>
-        <collision>thumb_distal_link_collision</collision>
+        <collision>link_thumb_3_collision</collision>
         <topic>prosthesis/sensor/thumb_fsr</topic>
       </contact>
@@ -250,5 +310,5 @@
     </sensor>
   </gazebo>
-  <gazebo reference="joint_middle_mcp">
+  <gazebo reference="joint_middle_1">
     <sensor name="prosthesis/sensor/middle_ft" type="force_torque">
       <always_on>true</always_on>
@@ -259,5 +319,5 @@
     </sensor>
   </gazebo>
-  <gazebo reference="joint_ring_mcp">
+  <gazebo reference="joint_ring_1">
     <sensor name="prosthesis/sensor/ring_ft" type="force_torque">
       <always_on>true</always_on>
@@ -268,5 +328,5 @@
     </sensor>
   </gazebo>
-  <gazebo reference="joint_little_mcp">
+  <gazebo reference="joint_little_1">
     <sensor name="prosthesis/sensor/little_ft" type="force_torque">
       <always_on>true</always_on>
@@ -277,5 +337,5 @@
     </sensor>
   </gazebo>
-  <gazebo reference="joint_thumb_cmc">
+  <gazebo reference="joint_thumb_1">
     <sensor name="prosthesis/sensor/thumb_ft" type="force_torque">
       <always_on>true</always_on>

File: ros2_ws/src/prosthesis_description/model/parameters.xacro (robot description, xacro)
@@ -10,25 +10,10 @@
     <xacro:property name="palm_width" value="0.098" />
     <xacro:property name="palm_depth" value="0.019" />
-    <xacro:property name="index_proximal_length" value="0.025" />
-    <xacro:property name="index_proximal_width" value="0.015" />
-    <xacro:property name="index_proximal_depth" value="0.012" />
-    <xacro:property name="index_middle_length" value="0.05" />
-    <xacro:property name="index_middle_width" value="0.015" />
-    <xacro:property name="index_middle_depth" value="0.012" />
-    <xacro:property name="middle_proximal_length" value="0.025" />
-    <xacro:property name="middle_proximal_width" value="0.015" />
-    <xacro:property name="middle_proximal_depth" value="0.012" />
-    <xacro:property name="ring_proximal_length" value="0.025" />
-    <xacro:property name="ring_proximal_width" value="0.015" />
-    <xacro:property name="ring_proximal_depth" value="0.012" />
-    <xacro:property name="ring_middle_length" value="0.05" />
-    <xacro:property name="ring_middle_width" value="0.015" />
-    <xacro:property name="ring_middle_depth" value="0.012" />
-    <xacro:property name="little_proximal_length" value="0.025" />
-    <xacro:property name="little_proximal_width" value="0.015" />
-    <xacro:property name="little_proximal_depth" value="0.012" />
-    <xacro:property name="little_middle_length" value="0.05" />
-    <xacro:property name="little_middle_width" value="0.015" />
-    <xacro:property name="little_middle_depth" value="0.012" />
+    <xacro:property name="finger_proximal_length" value="0.025" />
+    <xacro:property name="finger_proximal_width" value="0.015" />
+    <xacro:property name="finger_proximal_depth" value="0.012" />
+    <xacro:property name="finger_middle_length" value="0.05" />
+    <xacro:property name="finger_middle_width" value="0.015" />
+    <xacro:property name="finger_middle_depth" value="0.012" />
     <xacro:property name="thumb_metacarpal_length" value="0.01" />
     <xacro:property name="thumb_metacarpal_width" value="0.015" />
@@ -42,5 +27,5 @@
     <!-- MCP X and Y positions for each finger relative to palm_link -->
     <xacro:property name="mcp_x" value="${palm_length}" />
-    <xacro:property name="finger_width" value="${index_proximal_length}" />
+    <xacro:property name="finger_width" value="${finger_proximal_width}" />
     <xacro:property name="spacing_area" value="${palm_width - finger_width * 4}"/>
     <xacro:property name="d" value="${spacing_area / 5}"/>
