Commit message: Added clamping positions to trajectory_control.py

File: ros2_ws/src/prosthesis_description/model/gazebo.xacro (robot description, xacro)
@@ -250,10 +250,10 @@
   </gazebo>
   <!-- FSR -->
-  <gazebo reference="index_middle_fsr_link">
+  <gazebo reference="link_index_4">
     <sensor name="index_fsr" type="contact">
       <always_on>true</always_on>
       <update_rate>100</update_rate>
       <contact>
-        <collision>index_middle_fsr_link_collision</collision>
+        <collision>link_index_4_collision</collision>
         <topic>prosthesis/sensor/index_fsr</topic>
       </contact>
