Commit message: Improved trajectory_control (uses joint_states_broadcaster)

File: ros2_ws/src/prosthesis_description/model/gazebo.xacro (robot description, xacro)
@@ -13,9 +13,12 @@
     </plugin>
   </gazebo>
-  <gazebo>
+  <!--<gazebo>
       <plugin
           filename="gz-sim-joint-state-publisher-system"
           name="gz::sim::systems::JointStatePublisher">
           <topic>joint_states</topic>
+          <joint_name>joint_world_to_base_x</joint_name>
+          <joint_name>joint_base_x_to_base_y</joint_name>
+          <joint_name>joint_base_y_to_base_z</joint_name>
           <joint_name>joint_wrist_to_palm</joint_name>
           <joint_name>joint_index_1</joint_name>
@@ -39,5 +42,5 @@
           <joint_name>joint_thumb_3</joint_name>
       </plugin>
-    </gazebo>
+    </gazebo>-->
   <!-- Base and palm Gazebo tags -->
   <gazebo reference="base_link">
@@ -244,57 +247,59 @@
   <!-- IMU -->
   <gazebo reference="palm_link">
-    <sensor name="imu_sensor" type="imu">
+    <sensor name="prosthesis/sensor/palm_imu" type="imu">
       <always_on>true</always_on>
       <update_rate>50</update_rate>
+      <pose>0 0 0 0 0 0</pose>
+      <topic>/prosthesis/sensor/palm_imu</topic>
     </sensor>
   </gazebo>
   <!-- FSR -->
   <gazebo reference="link_index_4">
-    <sensor name="index_fsr" type="contact">
+    <sensor name="prosthesis/sensor/index_fsr" type="contact">
       <always_on>true</always_on>
       <update_rate>100</update_rate>
       <contact>
         <collision>link_index_4_collision</collision>
-        <topic>prosthesis/sensor/index_fsr</topic>
+        <topic>/prosthesis/sensor/index_fsr</topic>
       </contact>
     </sensor>
   </gazebo>
   <gazebo reference="link_middle_4">
-      <sensor name="middle_fsr" type="contact">
+      <sensor name="prosthesis/sensor/middle_fsr" type="contact">
       <always_on>true</always_on>
       <update_rate>100</update_rate>
       <contact>
         <collision>link_middle_4_collision</collision>
-        <topic>prosthesis/sensor/middle_fsr</topic>
+        <topic>/prosthesis/sensor/middle_fsr</topic>
       </contact>
     </sensor>
   </gazebo>
   <gazebo reference="link_ring_4">
-    <sensor name="ring_fsr" type="contact">
+    <sensor name="prosthesis/sensor/ring_fsr" type="contact">
       <always_on>true</always_on>
       <update_rate>100</update_rate>
       <contact>
         <collision>link_ring_4_collision</collision>
-        <topic>prosthesis/sensor/ring_fsr</topic>
+        <topic>/prosthesis/sensor/ring_fsr</topic>
       </contact>
     </sensor>
   </gazebo>
   <gazebo reference="link_little_4">
-    <sensor name="little_fsr" type="contact">
+    <sensor name="prosthesis/sensor/little_fsr" type="contact">
       <always_on>true</always_on>
       <update_rate>100</update_rate>
       <contact>
         <collision>link_little_4_collision</collision>
-        <topic>prosthesis/sensor/little_fsr</topic>
+        <topic>/prosthesis/sensor/little_fsr</topic>
       </contact>
     </sensor>
   </gazebo>
   <gazebo reference="link_thumb_3">
-    <sensor name="thumb_fsr" type="contact">
+    <sensor name="prosthesis/sensor/thumb_fsr" type="contact">
       <always_on>true</always_on>
       <update_rate>100</update_rate>
       <contact>
         <collision>link_thumb_3_collision</collision>
-        <topic>prosthesis/sensor/thumb_fsr</topic>
+        <topic>/prosthesis/sensor/thumb_fsr</topic>
       </contact>
     </sensor>
@@ -306,5 +311,5 @@
       <update_rate>100</update_rate>
       <pose>0 0 0 0 0 0</pose>
-      <topic>/index_ft</topic>
+      <topic>/prosthesis/sensor/index_ft</topic>
       <force_torque></force_torque>
     </sensor>
@@ -315,5 +320,5 @@
       <update_rate>100</update_rate>
       <pose>0 0 0 0 0 0</pose>
-      <topic>/middle_ft</topic>
+      <topic>/prosthesis/sensor/middle_ft</topic>
       <force_torque></force_torque>
     </sensor>
@@ -324,5 +329,5 @@
       <update_rate>100</update_rate>
       <pose>0 0 0 0 0 0</pose>
-      <topic>/ring_ft</topic>
+      <topic>/prosthesis/sensor/ring_ft</topic>
       <force_torque></force_torque>
     </sensor>
@@ -333,5 +338,5 @@
       <update_rate>100</update_rate>
       <pose>0 0 0 0 0 0</pose>
-      <topic>/little_ft</topic>
+      <topic>/prosthesis/sensor/little_ft</topic>
       <force_torque></force_torque>
     </sensor>
@@ -342,5 +347,5 @@
       <update_rate>100</update_rate>
       <pose>0 0 0 0 0 0</pose>
-      <topic>/thumb_ft</topic>
+      <topic>/prosthesis/sensor/thumb_ft</topic>
       <force_torque></force_torque>
     </sensor>

File: ros2_ws/src/prosthesis_description/model/prosthesis.urdf.xacro (robot description, xacro)
@@ -372,5 +372,5 @@
           <child link="base_link_x_frame"/>
           <axis xyz="1 0 0"/>
-          <limit lower="-2.0" upper="2.0" effort="100" velocity="1.0"/>
+          <limit lower="-1000" upper="1000" effort="100" velocity="1.0"/>
     </joint>
     <!-- Base X → Base Y (prismatic joint for y-axis motion) -->
@@ -380,5 +380,5 @@
           <child link="base_link_y_frame"/>
           <axis xyz="0 1 0"/>
-          <limit lower="-2.0" upper="2.0" effort="100" velocity="1.0"/>
+          <limit lower="-1000" upper="1000" effort="100" velocity="1.0"/>
     </joint>
     <!-- Base Y → Base Link (prismatic joint for z-axis motion) -->
@@ -388,5 +388,5 @@
           <child link="base_link"/>
           <axis xyz="0 0 1"/>
-          <limit lower="0.0" upper="2.0" effort="100" velocity="1.0"/>
+          <limit lower="0.0" upper="1000" effort="100" velocity="1.0"/>
     </joint>
     <!-- Base → Wrist -->
@@ -424,5 +424,5 @@
       <child link="link_index_3"/>
       <origin xyz="0.02 0.0025 0.0133" rpy="0 0 0"/><axis xyz="0 1 0"/>
-      <limit lower="0.0" upper="0.79" effort="2" velocity="5"/>
+      <limit lower="0.0" upper="1.57" effort="2" velocity="5"/>
     </joint>
     <joint name="joint_index_4" type="revolute">
