Commit message: Improved prosthesis movements, no more action use for joint trajectory controller

File: ros2_ws/src/prosthesis_description/model/gazebo.xacro (robot description, xacro)
@@ -14,5 +14,5 @@
   </gazebo>
   <!-- Base and palm Gazebo tags -->
-  <gazebo reference="base_link">
+  <gazebo reference="link_base_z">
     <material>Gazebo/Gray</material> <!-- Visual material used in Gazebo GUI -->
     <mu1>${base_wrist_friction}</mu1> <!-- Friction coefficients -->
@@ -23,12 +23,4 @@
     <maxVel>${max_velocity_default}</maxVel> <!-- Maximum velocity for contact -->
   </gazebo>
-  <gazebo reference="wrist_link">
-    <material>Gazebo/White</material>
-    <mu1>${base_wrist_friction}</mu1>
-    <mu2>${base_wrist_friction}</mu2>
-    <kp>${rigid_stiffness_default}</kp>
-    <kd>${damping_default}</kd>
-    <minDepth>${min_depth_default}</minDepth>
-  </gazebo>
   <gazebo reference="palm_link">
     <material>Gazebo/Orange</material>
@@ -152,5 +144,5 @@
   </gazebo>
   <!-- Thumb Gazebo tags -->
-  <gazebo reference="link_thumb_1">
+  <gazebo reference="link_thumb_1_x">
     <material>Gazebo/Blue</material>
     <mu1>${palm_fingers_friction}</mu1>
@@ -229,5 +221,5 @@
     </sensor>
   </gazebo>
-  <gazebo reference="link_thumb_3">
+  <gazebo reference="link_thumb_3_x">
     <sensor name="prosthesis/sensor/thumb_fsr" type="contact">
       <always_on>true</always_on>
@@ -285,5 +277,5 @@
     </sensor>
   </gazebo>
-  <gazebo reference="joint_thumb_1">
+  <gazebo reference="joint_thumb_1_x">
     <sensor name="prosthesis/sensor/thumb_ft" type="force_torque">
       <always_on>true</always_on>

File: ros2_ws/src/prosthesis_description/model/prosthesis.urdf.xacro (robot description, xacro)
@@ -8,5 +8,5 @@
     <link name="world" />
     <!-- Intermediate kinematic links for base movement (x, y, z) -->
-    <link name="base_link_x_frame">
+    <link name="link_base_x">
       <inertial>
         <mass value="0.001"/>
@@ -14,5 +14,5 @@
       </inertial>
     </link>
-    <link name="base_link_y_frame">
+    <link name="link_base_y">
       <inertial>
         <mass value="0.001"/>
@@ -20,5 +20,5 @@
       </inertial>
     </link>
-    <link name="base_link">
+    <link name="link_base_z">
       <visual>
           <origin xyz="0 0 0" rpy="0 0 1.53"/>
@@ -34,5 +34,5 @@
     </link>
     <xacro:property name="wrist_radius" value="0.01" />
-    <link name="wrist_link">
+    <link name="link_wrist_x">
       <collision>
           <origin xyz="${wrist_radius} 0 0" rpy="0 0 0"/>
@@ -43,4 +43,9 @@
       </xacro:inertial_sphere>
     </link>
+    <link name="link_wrist_y">
+      <xacro:inertial_sphere mass="0.2" radius="${wrist_radius}">
+          <origin xyz="${wrist_radius} 0 0" rpy="0 0 0"/>
+      </xacro:inertial_sphere>
+    </link>
     <link name="palm_link">
       <visual>
@@ -270,5 +275,5 @@
     </link>
     <!-- Thumb -->
-    <link name="link_thumb_1">
+    <link name="link_thumb_1_x">
       <visual>
           <origin xyz="0 0 0" rpy="0 1.57 0"/>
@@ -283,4 +288,9 @@
       </xacro:inertial_box>
     </link>
+    <link name="link_thumb_1_y">
+      <xacro:inertial_box mass="0.01" x="${thumb_metacarpal_length}" y="${thumb_metacarpal_width}" z="${thumb_metacarpal_depth}">
+          <origin xyz="0 0 0" rpy="0 0 0"/>
+      </xacro:inertial_box>
+    </link>
     <link name="link_thumb_2">
       <visual>
@@ -311,24 +321,24 @@
     <!-- ===== JOINTS ===== -->
     <!-- World → Base X (prismatic joint for x-axis motion) -->
-    <joint name="joint_world_to_base_x" type="prismatic">
+    <joint name="joint_base_x" type="prismatic">
           <origin xyz="0 0 0" rpy="0 0 0"/>
           <parent link="world"/>
-          <child link="base_link_x_frame"/>
+          <child link="link_base_x"/>
           <axis xyz="1 0 0"/>
           <limit lower="-1000" upper="1000" effort="100" velocity="1.0"/>
     </joint>
     <!-- Base X → Base Y (prismatic joint for y-axis motion) -->
-    <joint name="joint_base_x_to_base_y" type="prismatic">
-          <origin xyz="0 0 0" rpy="0 0 0"/>
-          <parent link="base_link_x_frame"/>
-          <child link="base_link_y_frame"/>
+    <joint name="joint_base_y" type="prismatic">
+          <origin xyz="0 0 0" rpy="0 0 0"/>
+          <parent link="link_base_x"/>
+          <child link="link_base_y"/>
           <axis xyz="0 1 0"/>
           <limit lower="-1000" upper="1000" effort="100" velocity="1.0"/>
     </joint>
     <!-- Base Y → Base Link (prismatic joint for z-axis motion) -->
-    <joint name="joint_base_y_to_base_z" type="prismatic">
-          <origin xyz="0 0 0" rpy="0 0 0"/>
-          <parent link="base_link_y_frame"/>
-          <child link="base_link"/>
+    <joint name="joint_base_z" type="prismatic">
+          <origin xyz="0 0 0" rpy="0 0 0"/>
+          <parent link="link_base_y"/>
+          <child link="link_base_z"/>
           <axis xyz="0 0 1"/>
           <limit lower="0.0" upper="1000" effort="100" velocity="1.0"/>
@@ -336,15 +346,21 @@
     <!-- Base → Wrist -->
     <joint name="joint_base_to_wrist" type="fixed">
-      <parent link="base_link"/>
-      <child  link="wrist_link"/>
+      <parent link="link_base_z"/>
+      <child  link="link_wrist_x"/>
       <origin xyz="0 0 ${wrist_radius}" rpy="0 0 0"/>
     </joint>
     <!-- Wrist → Palm -->
-    <joint name="joint_wrist_to_palm" type="revolute">
-      <parent link="wrist_link"/>
-      <child  link="palm_link"/>
+    <joint name="joint_wrist_x" type="revolute">
+      <parent link="link_wrist_x"/>
+      <child  link="link_wrist_y"/>
       <origin xyz="${wrist_radius*2} 0 0" rpy="0 0 0"/>
       <axis xyz="1 0 0"/>
-      <axis xyz="0 0 1"/>
+      <limit lower="-1.57" upper="1.57" effort="5" velocity="5"/>
+    </joint>
+    <joint name="joint_wrist_y" type="revolute">
+      <parent link="link_wrist_y"/>
+      <child  link="palm_link"/>
+      <origin xyz="0 0 0" rpy="0 0 0"/>
+      <axis xyz="0 1 0"/>
       <limit lower="-1.57" upper="1.57" effort="5" velocity="5"/>
     </joint>
@@ -430,12 +446,17 @@
       <limit lower="0.0" upper="1.57" effort="2" velocity="5"/>
     </joint>
-    <!-- Thumb (diagonal) -->
-    <joint name="joint_thumb_1" type="revolute">
-      <parent link="palm_link"/><child link="link_thumb_1"/>
+    <!-- Thumb -->
+    <joint name="joint_thumb_1_x" type="revolute">
+      <parent link="palm_link"/><child link="link_thumb_1_x"/>
       <origin xyz="0.05 0.04 0.001" rpy="0 0 0"/><axis xyz="-1 0 0"/>
       <limit lower="0" upper="1.57" effort="3" velocity="5"/>
     </joint>
+    <joint name="joint_thumb_1_y" type="revolute">
+      <parent link="link_thumb_1_x"/><child link="link_thumb_1_y"/>
+      <origin xyz="0 0 0" rpy="0 0 0"/><axis xyz="0 -1 0"/>
+      <limit lower="0" upper="1.57" effort="3" velocity="5"/>
+    </joint>
     <joint name="joint_thumb_2" type="revolute">
-      <parent link="link_thumb_1"/><child link="link_thumb_2"/>
+      <parent link="link_thumb_1_y"/><child link="link_thumb_2"/>
       <origin xyz="-0.0055 -0.003 -0.016" rpy="0 0 0"/><axis xyz="0 -1 0"/>
       <limit lower="0.0" upper="1.57" effort="2" velocity="5"/>
@@ -443,5 +464,5 @@
     <joint name="joint_thumb_3" type="revolute">
       <parent link="link_thumb_2"/><child link="link_thumb_3"/>
-      <origin xyz="-0.003 0.009 -0.04" rpy="0 0 0"/><axis xyz="0 1 0"/>
+      <origin xyz="-0.003 0.009 -0.04" rpy="0 0 0"/><axis xyz="0 -1 0"/>
       <limit lower="0.0" upper="1.57" effort="2" velocity="5"/>
     </joint>
@@ -454,17 +475,17 @@
     </hardware>
     <!-- Base Movement Joints (X, Y, Z) -->
-    <joint name="joint_world_to_base_x">
-      <command_interface name="position"/>
-      <state_interface name="position"/>
-      <state_interface name="velocity"/>
-      <state_interface name="effort"/>
-    </joint>
-    <joint name="joint_base_x_to_base_y">
-      <command_interface name="position"/>
-      <state_interface name="position"/>
-      <state_interface name="velocity"/>
-      <state_interface name="effort"/>
-    </joint>
-    <joint name="joint_base_y_to_base_z">
+    <joint name="joint_base_x">
+      <command_interface name="position"/> <!-- command controller will send for position control -->
+      <state_interface name="position"/>  <!-- state controller can read -->
+      <state_interface name="velocity"/>
+      <state_interface name="effort"/>
+    </joint>
+    <joint name="joint_base_y">
+      <command_interface name="position"/>
+      <state_interface name="position"/>
+      <state_interface name="velocity"/>
+      <state_interface name="effort"/>
+    </joint>
+    <joint name="joint_base_z">
       <command_interface name="position"/>
       <state_interface name="position"/>
@@ -473,7 +494,13 @@
     </joint>
     <!-- Wrist Joint -->
-    <joint name="joint_wrist_to_palm">
-      <command_interface name="position"/> <!-- command controller will send for position control -->
-      <state_interface name="position"/> <!-- state controller can read -->
+    <joint name="joint_wrist_x">
+      <command_interface name="position"/>
+      <state_interface name="position"/>
+      <state_interface name="velocity"/>
+      <state_interface name="effort"/>
+    </joint>
+    <joint name="joint_wrist_y">
+      <command_interface name="position"/>
+      <state_interface name="position"/>
       <state_interface name="velocity"/>
       <state_interface name="effort"/>
@@ -556,5 +583,11 @@
     </joint>
     <!-- Thumb Joints -->
-    <joint name="joint_thumb_1">
+    <joint name="joint_thumb_1_x">
+      <command_interface name="position"/>
+      <state_interface name="position"/>
+      <state_interface name="velocity"/>
+      <state_interface name="effort"/>
+    </joint>
+    <joint name="joint_thumb_1_y">
       <command_interface name="position"/>
       <state_interface name="position"/>

Commit message: Added scripts for dynamic CV stl spawner and movement of the arm toward the object

File: ros2_ws/src/prosthesis_description/model/gazebo.xacro (robot description, xacro)
@@ -14,5 +14,5 @@
   </gazebo>
   <!-- Base and palm Gazebo tags -->
-  <gazebo reference="link_base_z">
+  <gazebo reference="link_base_roll">
     <material>Gazebo/Gray</material> <!-- Visual material used in Gazebo GUI -->
     <mu1>${base_wrist_friction}</mu1> <!-- Friction coefficients -->

File: ros2_ws/src/prosthesis_description/model/prosthesis.urdf.xacro (robot description, xacro)
@@ -21,4 +21,10 @@
     </link>
     <link name="link_base_z">
+      <inertial>
+        <mass value="0.001"/>
+        <inertia ixx="0.0001" ixy="0.0" ixz="0.0" iyy="0.0001" iyz="0.0" izz="0.0001"/>
+      </inertial>
+    </link>
+    <link name="link_base_roll">
       <visual>
           <origin xyz="0 0 0" rpy="0 0 1.53"/>
@@ -29,11 +35,6 @@
           <geometry><mesh filename="$(find prosthesis_description)/meshes/forearm_final.stl"/></geometry>
       </collision>
-      <xacro:inertial_box mass="1.0" x="${base_length}" y="${base_width}" z="${base_depth}">
-          <origin xyz="0 0 0" rpy="0 0 0"/>
-      </xacro:inertial_box>
-    </link>
-    <link name="link_base_roll">
       <inertial>
-        <mass value="0.001"/>
+        <mass value="1.0"/>
         <inertia ixx="0.0001" ixy="0.0" ixz="0.0" iyy="0.0001" iyz="0.0" izz="0.0001"/>
       </inertial>
@@ -362,31 +363,31 @@
           <limit lower="-1000" upper="1000" effort="100" velocity="4"/>
     </joint>
-    <!-- Base R → Base Link (revolute joint for roll motion) -->
+    <!-- Base Y → Base Link (revolute joint for yaw motion - applied first for world frame) -->
+    <joint name="joint_base_yaw" type="revolute">
+          <origin xyz="0 0 0" rpy="0 0 0"/>
+          <parent link="link_base_z"/>
+          <child link="link_base_yaw"/>
+          <axis xyz="0 0 1"/>
+          <limit lower="-1.57" upper="1.57" effort="100" velocity="4"/>
+    </joint>
+    <!-- Base P → Base Link (revolute joint for pitch motion - applied second for world frame) -->
+    <joint name="joint_base_pitch" type="revolute">
+          <origin xyz="0 0 0" rpy="0 0 0"/>
+          <parent link="link_base_yaw"/>
+          <child link="link_base_pitch"/>
+          <axis xyz="0 1 0"/>
+          <limit lower="-1.57" upper="1.57" effort="100" velocity="4"/>
+    </joint>
+    <!-- Base R → Base Link (revolute joint for roll motion - applied last for world frame) -->
     <joint name="joint_base_roll" type="revolute">
           <origin xyz="0 0 0" rpy="0 0 0"/>
-          <parent link="link_base_z"/>
+          <parent link="link_base_pitch"/>
           <child link="link_base_roll"/>
           <axis xyz="1 0 0"/>
           <limit lower="-1.57" upper="1.57" effort="100" velocity="4"/>
     </joint>
-    <!-- Base P → Base Link (revolute joint for pitch motion) -->
-    <joint name="joint_base_pitch" type="revolute">
-          <origin xyz="0 0 0" rpy="0 0 0"/>
-          <parent link="link_base_roll"/>
-          <child link="link_base_pitch"/>
-          <axis xyz="0 1 0"/>
-          <limit lower="-1.57" upper="1.57" effort="100" velocity="4"/>
-    </joint>
-    <!-- Base Y → Base Link (revolute joint for yaw motion) -->
-    <joint name="joint_base_yaw" type="revolute">
-          <origin xyz="0 0 0" rpy="0 0 0"/>
-          <parent link="link_base_pitch"/>
-          <child link="link_base_yaw"/>
-          <axis xyz="0 0 1"/>
-          <limit lower="-1.57" upper="1.57" effort="100" velocity="4"/>
-    </joint>
     <!-- Base → Wrist -->
     <joint name="joint_base_to_wrist" type="fixed">
-      <parent link="link_base_yaw"/>
+      <parent link="link_base_roll"/>
       <child  link="link_wrist_x"/>
       <origin xyz="0 0 ${wrist_radius}" rpy="0 0 0"/>

Commit message: Added boxes for collision of the links, changed prosthesis colors

File: ros2_ws/src/prosthesis_description/model/gazebo.xacro (robot description, xacro)
@@ -15,5 +15,5 @@
   <!-- Base and palm Gazebo tags -->
   <gazebo reference="link_base_roll">
-    <material>Gazebo/Gray</material> <!-- Visual material used in Gazebo GUI -->
+    <material>Gazebo/Black</material> <!-- Visual material used in Gazebo GUI -->
     <mu1>${base_wrist_friction}</mu1> <!-- Friction coefficients -->
     <mu2>${base_wrist_friction}</mu2>
@@ -24,5 +24,5 @@
   </gazebo>
   <gazebo reference="palm_link">
-    <material>Gazebo/Orange</material>
+    <material>Gazebo/Black</material>
     <mu1>${palm_fingers_friction}</mu1>
     <mu2>${palm_fingers_friction}</mu2>
@@ -33,5 +33,5 @@
   <!-- Index finger Gazebo tags -->
   <gazebo reference="link_index_1">
-    <material>Gazebo/Blue</material>
+    <material>Gazebo/Gray</material>
     <mu1>${palm_fingers_friction}</mu1>
     <mu2>${palm_fingers_friction}</mu2>
@@ -42,5 +42,5 @@
   </gazebo>
   <gazebo reference="link_index_2">
-    <material>Gazebo/Red</material>
+    <material>Gazebo/Gray</material>
     <mu1>${palm_fingers_friction}</mu1>
     <mu2>${palm_fingers_friction}</mu2>
@@ -51,5 +51,5 @@
   </gazebo>
   <gazebo reference="link_index_3">
-    <material>Gazebo/Blue</material>
+    <material>Gazebo/Orange</material>
     <mu1>${palm_fingers_friction}</mu1>
     <mu2>${palm_fingers_friction}</mu2>
@@ -61,5 +61,5 @@
   <!-- Middle finger Gazebo tags -->
   <gazebo reference="link_middle_1">
-    <material>Gazebo/Blue</material>
+    <material>Gazebo/Gray</material>
     <mu1>${palm_fingers_friction}</mu1>
     <mu2>${palm_fingers_friction}</mu2>
@@ -70,5 +70,5 @@
   </gazebo>
   <gazebo reference="link_middle_2">
-    <material>Gazebo/Red</material>
+    <material>Gazebo/Gray</material>
     <mu1>${palm_fingers_friction}</mu1>
     <mu2>${palm_fingers_friction}</mu2>
@@ -79,5 +79,5 @@
   </gazebo>
   <gazebo reference="link_middle_3">
-    <material>Gazebo/Blue</material>
+    <material>Gazebo/Orange</material>
     <mu1>${palm_fingers_friction}</mu1>
     <mu2>${palm_fingers_friction}</mu2>
@@ -89,5 +89,5 @@
   <!-- Ring finger Gazebo tags -->
   <gazebo reference="link_ring_1">
-    <material>Gazebo/Blue</material>
+    <material>Gazebo/Gray</material>
     <mu1>${palm_fingers_friction}</mu1>
     <mu2>${palm_fingers_friction}</mu2>
@@ -98,5 +98,5 @@
   </gazebo>
   <gazebo reference="link_ring_2">
-    <material>Gazebo/Red</material>
+    <material>Gazebo/Gray</material>
     <mu1>${palm_fingers_friction}</mu1>
     <mu2>${palm_fingers_friction}</mu2>
@@ -107,5 +107,5 @@
   </gazebo>
   <gazebo reference="link_ring_3">
-    <material>Gazebo/Blue</material>
+    <material>Gazebo/Orange</material>
     <mu1>${palm_fingers_friction}</mu1>
     <mu2>${palm_fingers_friction}</mu2>
@@ -117,5 +117,5 @@
   <!-- Little finger Gazebo tags -->
   <gazebo reference="link_little_1">
-    <material>Gazebo/Blue</material>
+    <material>Gazebo/Gray</material>
     <mu1>${palm_fingers_friction}</mu1>
     <mu2>${palm_fingers_friction}</mu2>
@@ -126,5 +126,5 @@
   </gazebo>
   <gazebo reference="link_little_2">
-    <material>Gazebo/Red</material>
+    <material>Gazebo/Gray</material>
     <mu1>${palm_fingers_friction}</mu1>
     <mu2>${palm_fingers_friction}</mu2>
@@ -135,5 +135,5 @@
   </gazebo>
   <gazebo reference="link_little_3">
-    <material>Gazebo/Blue</material>
+    <material>Gazebo/Orange</material>
     <mu1>${palm_fingers_friction}</mu1>
     <mu2>${palm_fingers_friction}</mu2>
@@ -145,5 +145,5 @@
   <!-- Thumb Gazebo tags -->
   <gazebo reference="link_thumb_1_x">
-    <material>Gazebo/Blue</material>
+    <material>Gazebo/Black</material>
     <mu1>${palm_fingers_friction}</mu1>
     <mu2>${palm_fingers_friction}</mu2>
@@ -154,5 +154,5 @@
   </gazebo>
   <gazebo reference="link_thumb_2">
-    <material>Gazebo/Red</material>
+    <material>Gazebo/Gray</material>
     <mu1>${palm_fingers_friction}</mu1>
     <mu2>${palm_fingers_friction}</mu2>
@@ -163,5 +163,5 @@
   </gazebo>
   <gazebo reference="link_thumb_3">
-    <material>Gazebo/Blue</material>
+    <material>Gazebo/Orange</material>
     <mu1>${palm_fingers_friction}</mu1>
     <mu2>${palm_fingers_friction}</mu2>

File: ros2_ws/src/prosthesis_description/model/parameters.xacro (robot description, xacro)
@@ -4,25 +4,28 @@
     <!-- ==== PROSTHESIS VALUES ==== -->
     <!-- Dimensions for each link -->
-    <xacro:property name="base_length" value="0.174" />
-    <xacro:property name="base_width" value="0.065" />
-    <xacro:property name="base_depth" value="0.101" />
-    <xacro:property name="palm_length" value="0.068" />
-    <xacro:property name="palm_width" value="0.098" />
-    <xacro:property name="palm_depth" value="0.019" />
-    <xacro:property name="finger_proximal_length" value="0.025" />
+    <xacro:property name="base_length" value="0.19" />
+    <xacro:property name="base_width" value="0.069" />
+    <xacro:property name="base_depth" value="0.051" />
+    <xacro:property name="palm_length" value="0.092" />
+    <xacro:property name="palm_width" value="0.096" />
+    <xacro:property name="palm_depth" value="0.03" />
+    <xacro:property name="finger_proximal_length" value="0.028" />
     <xacro:property name="finger_proximal_width" value="0.015" />
-    <xacro:property name="finger_proximal_depth" value="0.012" />
-    <xacro:property name="finger_middle_length" value="0.05" />
+    <xacro:property name="finger_proximal_depth" value="0.015" />
+    <xacro:property name="finger_middle_length" value="0.02" />
     <xacro:property name="finger_middle_width" value="0.015" />
-    <xacro:property name="finger_middle_depth" value="0.012" />
+    <xacro:property name="finger_middle_depth" value="0.015" />
+    <xacro:property name="finger_distal_length" value="0.025" />
+    <xacro:property name="finger_distal_width" value="0.015" />
+    <xacro:property name="finger_distal_depth" value="0.015" />
     <xacro:property name="thumb_metacarpal_length" value="0.01" />
     <xacro:property name="thumb_metacarpal_width" value="0.015" />
-    <xacro:property name="thumb_metacarpal_depth" value="0.012" />
+    <xacro:property name="thumb_metacarpal_depth" value="0.015" />
     <xacro:property name="thumb_proximal_length" value="0.025" />
     <xacro:property name="thumb_proximal_width" value="0.015" />
-    <xacro:property name="thumb_proximal_depth" value="0.012" />
+    <xacro:property name="thumb_proximal_depth" value="0.015" />
     <xacro:property name="thumb_distal_length" value="0.020" />
     <xacro:property name="thumb_distal_width" value="0.015" />
-    <xacro:property name="thumb_distal_depth" value="0.012" />
+    <xacro:property name="thumb_distal_depth" value="0.015" />
     <!-- MCP X and Y positions for each finger relative to palm_link -->
     <xacro:property name="mcp_x" value="${palm_length}" />
