Commit message: Added boxes for collision of the links, changed prosthesis colors

File: ros2_ws/src/prosthesis_description/model/prosthesis.urdf.xacro (robot description, xacro)
@@ -9,20 +9,17 @@
     <!-- Intermediate kinematic links for base movement (x, y, z) -->
     <link name="link_base_x">
-      <inertial>
-        <mass value="0.001"/>
-        <inertia ixx="0.0001" ixy="0.0" ixz="0.0" iyy="0.0001" iyz="0.0" izz="0.0001"/>
-      </inertial>
+      <xacro:inertial_box mass="0.1" x="${base_length}" y="${base_width}" z="${base_depth}">
+          <origin xyz="${-base_length} 0 ${base_depth/2}" rpy="0 0 0"/>
+      </xacro:inertial_box>
     </link>
     <link name="link_base_y">
-      <inertial>
-        <mass value="0.001"/>
-        <inertia ixx="0.0001" ixy="0.0" ixz="0.0" iyy="0.0001" iyz="0.0" izz="0.0001"/>
-      </inertial>
+      <xacro:inertial_box mass="0.1" x="${base_length}" y="${base_width}" z="${base_depth}">
+          <origin xyz="${-base_length} 0 ${base_depth/2}" rpy="0 0 0"/>
+      </xacro:inertial_box>
     </link>
     <link name="link_base_z">
-      <inertial>
-        <mass value="0.001"/>
-        <inertia ixx="0.0001" ixy="0.0" ixz="0.0" iyy="0.0001" iyz="0.0" izz="0.0001"/>
-      </inertial>
+      <xacro:inertial_box mass="0.1" x="${base_length}" y="${base_width}" z="${base_depth}">
+          <origin xyz="${-base_length} 0 ${base_depth/2}" rpy="0 0 0"/>
+      </xacro:inertial_box>
     </link>
     <link name="link_base_roll">
@@ -32,23 +29,20 @@
       </visual>
       <collision>
-          <origin xyz="0 0 0" rpy="0 0 1.53"/>
-          <geometry><mesh filename="$(find prosthesis_description)/meshes/forearm_final.stl"/></geometry>
-      </collision>
-      <inertial>
-        <mass value="1.0"/>
-        <inertia ixx="0.0001" ixy="0.0" ixz="0.0" iyy="0.0001" iyz="0.0" izz="0.0001"/>
-      </inertial>
+        <origin xyz="${-base_length/2} 0 ${base_depth/2}" rpy="0 0 0"/>
+        <geometry><box size="${base_length} ${base_width} ${base_depth}"/></geometry>
+      </collision>
+      <xacro:inertial_box mass="0.1" x="${base_length}" y="${base_width}" z="${base_depth}">
+          <origin xyz="${-base_length} 0 ${base_depth/2}" rpy="0 0 0"/>
+      </xacro:inertial_box>
     </link>
     <link name="link_base_pitch">
-      <inertial>
-        <mass value="0.001"/>
-        <inertia ixx="0.0001" ixy="0.0" ixz="0.0" iyy="0.0001" iyz="0.0" izz="0.0001"/>
-      </inertial>
+      <xacro:inertial_box mass="0.1" x="${base_length}" y="${base_width}" z="${base_depth}">
+          <origin xyz="${-base_length} 0 ${base_depth/2}" rpy="0 0 0"/>
+      </xacro:inertial_box>
     </link>
     <link name="link_base_yaw">
-      <inertial>
-        <mass value="0.001"/>
-        <inertia ixx="0.0001" ixy="0.0" ixz="0.0" iyy="0.0001" iyz="0.0" izz="0.0001"/>
-      </inertial>
+      <xacro:inertial_box mass="0.1" x="${base_length}" y="${base_width}" z="${base_depth}">
+          <origin xyz="${-base_length} 0 ${base_depth/2}" rpy="0 0 0"/>
+      </xacro:inertial_box>
     </link>
     <xacro:property name="wrist_radius" value="0.01" />
@@ -58,10 +52,10 @@
           <geometry><sphere radius="${wrist_radius}"/></geometry>
       </collision>
-      <xacro:inertial_sphere mass="0.2" radius="${wrist_radius}">
+      <xacro:inertial_sphere mass="0.05" radius="${wrist_radius}">
           <origin xyz="${wrist_radius} 0 0" rpy="0 0 0"/>
       </xacro:inertial_sphere>
     </link>
     <link name="link_wrist_y">
-      <xacro:inertial_sphere mass="0.2" radius="${wrist_radius}">
+      <xacro:inertial_sphere mass="0.05" radius="${wrist_radius}">
           <origin xyz="${wrist_radius} 0 0" rpy="0 0 0"/>
       </xacro:inertial_sphere>
@@ -69,13 +63,13 @@
     <link name="palm_link">
       <visual>
-          <origin xyz="0 0 0" rpy="1.57 3.14 -1.53"/>
-          <geometry><mesh filename="$(find prosthesis_description)/meshes/Palm_main_body.stl"/></geometry>
-      </visual>
-      <collision>
-          <origin xyz="0 0 0" rpy="1.57 3.14 -1.53"/>
-          <geometry><mesh filename="$(find prosthesis_description)/meshes/Palm_main_body.stl"/></geometry>
+        <origin xyz="0 0 0" rpy="1.57 3.14 -1.53"/>
+        <geometry><mesh filename="$(find prosthesis_description)/meshes/Palm_main_body.stl"/></geometry>
+      </visual>
+      <collision>
+        <origin xyz="${palm_length/2} 0 ${palm_depth/2}" rpy="0 0 0"/>
+        <geometry><box size="${palm_length} ${palm_width} ${palm_depth}"/></geometry>
       </collision>
       <xacro:inertial_box mass="0.2" x="${palm_length}" y="${palm_width}" z="${palm_depth}">
-          <origin xyz="${palm_length/2} 0 0" rpy="0 0 0"/>
+          <origin xyz="${palm_length} 0 ${palm_depth}" rpy="0 0 0"/>
       </xacro:inertial_box>
     </link>
@@ -88,9 +82,9 @@
       </visual>
       <collision>
-          <origin xyz="0 0 0" rpy="0 0 0"/>
-          <geometry><mesh filename="$(find prosthesis_description)/meshes/A_PhalangeConstruction_Part_3.stl"/></geometry>
+        <origin xyz="${finger_proximal_length/2} ${finger_proximal_width/2} ${-finger_proximal_depth/2}" rpy="0 0 0"/>
+        <geometry><box size="${finger_proximal_length} ${finger_proximal_width} ${finger_proximal_depth}"/></geometry>
       </collision>
       <xacro:inertial_box mass="0.01" x="${finger_proximal_length}" y="${finger_proximal_width}" z="${finger_proximal_depth}">
-          <origin xyz="${finger_proximal_length/2} 0 0" rpy="0 0 0"/>
+          <origin xyz="${finger_proximal_length} ${finger_proximal_width} ${-finger_proximal_depth}" rpy="0 0 0"/>
       </xacro:inertial_box>
     </link>
@@ -101,9 +95,9 @@
       </visual>
       <collision>
-          <origin xyz="0 0 0" rpy="0 0 0"/>
-          <geometry><mesh filename="$(find prosthesis_description)/meshes/A_PhalangeConstruction_Part_4.stl"/></geometry>
+        <origin xyz="${finger_middle_length/2 - 0.001} ${finger_middle_width/4} ${finger_middle_depth/2}" rpy="0 0 0"/>
+        <geometry><box size="${finger_middle_length} ${finger_middle_width} ${finger_middle_depth}"/></geometry>
       </collision>
       <xacro:inertial_box mass="0.02" x="${finger_middle_length}" y="${finger_middle_width}" z="${finger_middle_depth}">
-          <origin xyz="${finger_middle_length/2} 0 0" rpy="0 0 0"/>
+          <origin xyz="${finger_middle_length} ${finger_middle_width} ${finger_middle_depth}" rpy="0 0 0"/>
       </xacro:inertial_box>
     </link>
@@ -113,11 +107,4 @@
           <geometry><mesh filename="$(find prosthesis_description)/meshes/A_PhalangeConstruction_Part_4.stl"/></geometry>
       </visual>
-      <collision>
-          <origin xyz="0 0 0" rpy="0 0 0"/>
-          <geometry><mesh filename="$(find prosthesis_description)/meshes/A_PhalangeConstruction_Part_4.stl"/></geometry>
-      </collision>
-      <xacro:inertial_box mass="0.02" x="${finger_middle_length}" y="${finger_middle_width}" z="${finger_middle_depth}">
-          <origin xyz="${finger_middle_length/2} 0 0" rpy="0 0 0"/>
-      </xacro:inertial_box>
     </link>
     <link name="link_index_3">
@@ -127,52 +114,91 @@
       </visual>
       <collision>
+        <origin xyz="${finger_distal_length/2 + 0.001} 0 ${-finger_distal_depth/2}" rpy="0 0 0"/>
+        <geometry><box size="${finger_distal_length} ${finger_distal_width} ${finger_distal_depth}"/></geometry>
+      </collision>
+      <xacro:inertial_box mass="0.02" x="${finger_distal_length}" y="${finger_distal_width}" z="${finger_distal_depth}">
+          <origin xyz="${finger_distal_length} ${finger_distal_width/2} ${finger_distal_depth}" rpy="0 0 0"/>
+      </xacro:inertial_box>
+    </link>
+    <!-- Middle -->
+    <link name="link_middle_1">
+      <visual>
+          <origin xyz="0 0 0" rpy="0 0 0"/>
+          <geometry><mesh filename="$(find prosthesis_description)/meshes/A_PhalangeConstruction_Part_3.stl"/></geometry>
+      </visual>
+      <collision>
+        <origin xyz="${finger_proximal_length/2} ${finger_proximal_width/2} ${-finger_proximal_depth/2}" rpy="0 0 0"/>
+        <geometry><box size="${finger_proximal_length} ${finger_proximal_width} ${finger_proximal_depth}"/></geometry>
+      </collision>
+      <xacro:inertial_box mass="0.01" x="${finger_proximal_length}" y="${finger_proximal_width}" z="${finger_proximal_depth}">
+          <origin xyz="${finger_proximal_length} ${finger_proximal_width} ${-finger_proximal_depth}" rpy="0 0 0"/>
+      </xacro:inertial_box>
+    </link>
+    <link name="link_middle_2">
+      <visual>
+          <origin xyz="0 0 0" rpy="0 0 00"/>
+          <geometry><mesh filename="$(find prosthesis_description)/meshes/A_PhalangeConstruction_Part_4.stl"/></geometry>
+      </visual>
+      <collision>
+        <origin xyz="${finger_middle_length/2 - 0.001} ${finger_middle_width/4} ${finger_middle_depth/2}" rpy="0 0 0"/>
+        <geometry><box size="${finger_middle_length} ${finger_middle_width} ${finger_middle_depth}"/></geometry>
+      </collision>
+      <xacro:inertial_box mass="0.02" x="${finger_middle_length}" y="${finger_middle_width}" z="${finger_middle_depth}">
+          <origin xyz="${finger_middle_length} ${finger_middle_width} ${finger_middle_depth}" rpy="0 0 0"/>
+      </xacro:inertial_box>
+    </link>
+    <link name="link_middle_2_b">
+      <visual>
+          <origin xyz="0 0 0" rpy="0 0 0"/>
+          <geometry><mesh filename="$(find prosthesis_description)/meshes/A_PhalangeConstruction_Part_4.stl"/></geometry>
+      </visual>
+    </link>
+    <link name="link_middle_3">
+      <visual>
           <origin xyz="0 0 0" rpy="-1.57 0 1.57"/>
           <geometry><mesh filename="$(find prosthesis_description)/meshes/A_PhalangeConstruction_Part_6.stl"/></geometry>
+      </visual>
+      <collision>
+        <origin xyz="${finger_distal_length/2 + 0.001} 0 ${-finger_distal_depth/2}" rpy="0 0 0"/>
+        <geometry><box size="${finger_distal_length} ${finger_distal_width} ${finger_distal_depth}"/></geometry>
+      </collision>
+      <xacro:inertial_box mass="0.02" x="${finger_distal_length}" y="${finger_distal_width}" z="${finger_distal_depth}">
+          <origin xyz="${finger_distal_length} ${finger_distal_width/2} ${finger_distal_depth}" rpy="0 0 0"/>
+      </xacro:inertial_box>
+    </link>
+    <!-- Ring -->
+    <link name="link_ring_1">
+      <visual>
+          <origin xyz="0 0 0" rpy="0 0 0"/>
+          <geometry><mesh filename="$(find prosthesis_description)/meshes/A_PhalangeConstruction_Part_3.stl"/></geometry>
+      </visual>
+      <collision>
+        <origin xyz="${finger_proximal_length/2} ${finger_proximal_width/2} ${-finger_proximal_depth/2}" rpy="0 0 0"/>
+        <geometry><box size="${finger_proximal_length} ${finger_proximal_width} ${finger_proximal_depth}"/></geometry>
+      </collision>
+      <xacro:inertial_box mass="0.01" x="${finger_proximal_length}" y="${finger_proximal_width}" z="${finger_proximal_depth}">
+          <origin xyz="${finger_proximal_length} ${finger_proximal_width} ${-finger_proximal_depth}" rpy="0 0 0"/>
+      </xacro:inertial_box>
+    </link>
+    <link name="link_ring_2">
+      <visual>
+          <origin xyz="0 0 0" rpy="0 0 0"/>
+          <geometry><mesh filename="$(find prosthesis_description)/meshes/A_PhalangeConstruction_Part_4.stl"/></geometry>
+      </visual>
+      <collision>
+        <origin xyz="${finger_middle_length/2 - 0.001} ${finger_middle_width/4} ${finger_middle_depth/2}" rpy="0 0 0"/>
+        <geometry><box size="${finger_middle_length} ${finger_middle_width} ${finger_middle_depth}"/></geometry>
       </collision>
       <xacro:inertial_box mass="0.02" x="${finger_middle_length}" y="${finger_middle_width}" z="${finger_middle_depth}">
-          <origin xyz="${finger_middle_length/2} 0 0" rpy="0 0 0"/>
-      </xacro:inertial_box>
-    </link>
-    <!-- Middle -->
-    <link name="link_middle_1">
-      <visual>
-          <origin xyz="0 0 0" rpy="0 0 0"/>
-          <geometry><mesh filename="$(find prosthesis_description)/meshes/A_PhalangeConstruction_Part_3.stl"/></geometry>
-      </visual>
-      <collision>
-          <origin xyz="0 0 0" rpy="0 0 0"/>
-          <geometry><mesh filename="$(find prosthesis_description)/meshes/A_PhalangeConstruction_Part_3.stl"/></geometry>
-      </collision>
-      <xacro:inertial_box mass="0.01" x="${finger_proximal_length}" y="${finger_proximal_width}" z="${finger_proximal_depth}">
-          <origin xyz="${finger_proximal_length/2} 0 0" rpy="0 0 0"/>
-      </xacro:inertial_box>
-    </link>
-    <link name="link_middle_2">
-      <visual>
-          <origin xyz="0 0 0" rpy="0 0 00"/>
-          <geometry><mesh filename="$(find prosthesis_description)/meshes/A_PhalangeConstruction_Part_4.stl"/></geometry>
-      </visual>
-      <collision>
-          <origin xyz="0 0 0" rpy="0 0 0"/>
-          <geometry><mesh filename="$(find prosthesis_description)/meshes/A_PhalangeConstruction_Part_4.stl"/></geometry>
-      </collision>
-      <xacro:inertial_box mass="0.02" x="${finger_middle_length}" y="${finger_middle_width}" z="${finger_middle_depth}">
-          <origin xyz="${finger_middle_length/2} 0 0" rpy="0 0 0"/>
-      </xacro:inertial_box>
-    </link>
-    <link name="link_middle_2_b">
-      <visual>
-          <origin xyz="0 0 0" rpy="0 0 0"/>
-          <geometry><mesh filename="$(find prosthesis_description)/meshes/A_PhalangeConstruction_Part_4.stl"/></geometry>
-      </visual>
-      <collision>
-          <origin xyz="0 0 0" rpy="0 0 0"/>
-          <geometry><mesh filename="$(find prosthesis_description)/meshes/A_PhalangeConstruction_Part_4.stl"/></geometry>
-      </collision>
-      <xacro:inertial_box mass="0.02" x="${finger_middle_length}" y="${finger_middle_width}" z="${finger_middle_depth}">
-          <origin xyz="${finger_middle_length/2} 0 0" rpy="0 0 0"/>
-      </xacro:inertial_box>
-    </link>
-    <link name="link_middle_3">
+          <origin xyz="${finger_middle_length} ${finger_middle_width} ${finger_middle_depth}" rpy="0 0 0"/>
+      </xacro:inertial_box>
+    </link>
+    <link name="link_ring_2_b">
+      <visual>
+          <origin xyz="0 0 0" rpy="0 0 0"/>
+          <geometry><mesh filename="$(find prosthesis_description)/meshes/A_PhalangeConstruction_Part_4.stl"/></geometry>
+      </visual>
+    </link>
+    <link name="link_ring_3">
       <visual>
           <origin xyz="0 0 0" rpy="-1.57 0 1.57"/>
@@ -180,115 +206,55 @@
       </visual>
       <collision>
+        <origin xyz="${finger_distal_length/2 + 0.001} 0 ${-finger_distal_depth/2}" rpy="0 0 0"/>
+        <geometry><box size="${finger_distal_length} ${finger_distal_width} ${finger_distal_depth}"/></geometry>
+      </collision>
+      <xacro:inertial_box mass="0.02" x="${finger_distal_length}" y="${finger_distal_width}" z="${finger_distal_depth}">
+          <origin xyz="${finger_distal_length} ${finger_distal_width/2} ${finger_distal_depth}" rpy="0 0 0"/>
+      </xacro:inertial_box>
+    </link>
+    <!-- Little -->
+    <link name="link_little_1">
+      <visual>
+          <origin xyz="0 0 0" rpy="0 0 0"/>
+          <geometry><mesh filename="$(find prosthesis_description)/meshes/A_PhalangeConstruction_Part_3.stl"/></geometry>
+      </visual>
+      <collision>
+        <origin xyz="${finger_proximal_length/2} ${finger_proximal_width/2} ${-finger_proximal_depth/2}" rpy="0 0 0"/>
+        <geometry><box size="${finger_proximal_length} ${finger_proximal_width} ${finger_proximal_depth}"/></geometry>
+      </collision>
+      <xacro:inertial_box mass="0.01" x="${finger_proximal_length}" y="${finger_proximal_width}" z="${finger_proximal_depth}">
+          <origin xyz="${finger_proximal_length} ${finger_proximal_width} ${-finger_proximal_depth}" rpy="0 0 0"/>
+      </xacro:inertial_box>
+    </link>
+    <link name="link_little_2">
+      <visual>
+          <origin xyz="0 0 0" rpy="0 0 0"/>
+          <geometry><mesh filename="$(find prosthesis_description)/meshes/A_PhalangeConstruction_Part_4.stl"/></geometry>
+      </visual>
+      <collision>
+        <origin xyz="${finger_middle_length/2 - 0.001} ${finger_middle_width/4} ${finger_middle_depth/2}" rpy="0 0 0"/>
+        <geometry><box size="${finger_middle_length} ${finger_middle_width} ${finger_middle_depth}"/></geometry>
+      </collision>
+      <xacro:inertial_box mass="0.02" x="${finger_middle_length}" y="${finger_middle_width}" z="${finger_middle_depth}">
+          <origin xyz="${finger_middle_length} ${finger_middle_width} ${finger_middle_depth}" rpy="0 0 0"/>
+      </xacro:inertial_box>
+    </link>
+    <link name="link_little_2_b">
+      <visual>
+          <origin xyz="0 0 0" rpy="0 0 0"/>
+          <geometry><mesh filename="$(find prosthesis_description)/meshes/A_PhalangeConstruction_Part_4.stl"/></geometry>
+      </visual>
+    </link>
+    <link name="link_little_3">
+      <visual>
           <origin xyz="0 0 0" rpy="-1.57 0 1.57"/>
           <geometry><mesh filename="$(find prosthesis_description)/meshes/A_PhalangeConstruction_Part_6.stl"/></geometry>
-      </collision>
-      <xacro:inertial_box mass="0.02" x="${finger_middle_length}" y="${finger_middle_width}" z="${finger_middle_depth}">
-          <origin xyz="${finger_middle_length/2} 0 0" rpy="0 0 0"/>
-      </xacro:inertial_box>
-    </link>
-    <!-- Ring -->
-    <link name="link_ring_1">
-      <visual>
-          <origin xyz="0 0 0" rpy="0 0 0"/>
-          <geometry><mesh filename="$(find prosthesis_description)/meshes/A_PhalangeConstruction_Part_3.stl"/></geometry>
-      </visual>
-      <collision>
-          <origin xyz="0 0 0" rpy="0 0 0"/>
-          <geometry><mesh filename="$(find prosthesis_description)/meshes/A_PhalangeConstruction_Part_3.stl"/></geometry>
-      </collision>
-      <xacro:inertial_box mass="0.01" x="${finger_proximal_length}" y="${finger_proximal_width}" z="${finger_proximal_depth}">
-          <origin xyz="${finger_proximal_length/2} 0 0" rpy="0 0 0"/>
-      </xacro:inertial_box>
-    </link>
-    <link name="link_ring_2">
-      <visual>
-          <origin xyz="0 0 0" rpy="0 0 0"/>
-          <geometry><mesh filename="$(find prosthesis_description)/meshes/A_PhalangeConstruction_Part_4.stl"/></geometry>
-      </visual>
-      <collision>
-          <origin xyz="0 0 0" rpy="0 0 0"/>
-          <geometry><mesh filename="$(find prosthesis_description)/meshes/A_PhalangeConstruction_Part_4.stl"/></geometry>
-      </collision>
-      <xacro:inertial_box mass="0.02" x="${finger_middle_length}" y="${finger_middle_width}" z="${finger_middle_depth}">
-          <origin xyz="${finger_middle_length/2} 0 0" rpy="0 0 0"/>
-      </xacro:inertial_box>
-    </link>
-    <link name="link_ring_2_b">
-      <visual>
-          <origin xyz="0 0 0" rpy="0 0 0"/>
-          <geometry><mesh filename="$(find prosthesis_description)/meshes/A_PhalangeConstruction_Part_4.stl"/></geometry>
-      </visual>
-      <collision>
-          <origin xyz="0 0 0" rpy="0 0 0"/>
-          <geometry><mesh filename="$(find prosthesis_description)/meshes/A_PhalangeConstruction_Part_4.stl"/></geometry>
-      </collision>
-      <xacro:inertial_box mass="0.02" x="${finger_middle_length}" y="${finger_middle_width}" z="${finger_middle_depth}">
-          <origin xyz="${finger_middle_length/2} 0 0" rpy="0 0 0"/>
-      </xacro:inertial_box>
-    </link>
-    <link name="link_ring_3">
-      <visual>
-          <origin xyz="0 0 0" rpy="-1.57 0 1.57"/>
-          <geometry><mesh filename="$(find prosthesis_description)/meshes/A_PhalangeConstruction_Part_6.stl"/></geometry>
-      </visual>
-      <collision>
-          <origin xyz="0 0 0" rpy="-1.57 0 1.57"/>
-          <geometry><mesh filename="$(find prosthesis_description)/meshes/A_PhalangeConstruction_Part_6.stl"/></geometry>
-      </collision>
-      <xacro:inertial_box mass="0.02" x="${finger_middle_length}" y="${finger_middle_width}" z="${finger_middle_depth}">
-          <origin xyz="${finger_middle_length/2} 0 0" rpy="0 0 0"/>
-      </xacro:inertial_box>
-    </link>
-    <!-- Little -->
-    <link name="link_little_1">
-      <visual>
-          <origin xyz="0 0 0" rpy="0 0 0"/>
-          <geometry><mesh filename="$(find prosthesis_description)/meshes/A_PhalangeConstruction_Part_3.stl"/></geometry>
-      </visual>
-      <collision>
-          <origin xyz="0 0 0" rpy="0 0 0"/>
-          <geometry><mesh filename="$(find prosthesis_description)/meshes/A_PhalangeConstruction_Part_3.stl"/></geometry>
-      </collision>
-      <xacro:inertial_box mass="0.01" x="${finger_proximal_length}" y="${finger_proximal_width}" z="${finger_proximal_depth}">
-          <origin xyz="${finger_proximal_length/2} 0 0" rpy="0 0 0"/>
-      </xacro:inertial_box>
-    </link>
-    <link name="link_little_2">
-      <visual>
-          <origin xyz="0 0 0" rpy="0 0 0"/>
-          <geometry><mesh filename="$(find prosthesis_description)/meshes/A_PhalangeConstruction_Part_4.stl"/></geometry>
-      </visual>
-      <collision>
-          <origin xyz="0 0 0" rpy="0 0 0"/>
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